File: Hexapod/PWM.brd (EAGLE design)
At the start: 48.9 x 39.6 mm, 44 parts, among them IC1 AT32UC3L016/32/64, IC2 TXS0108ERGYRGY, IC3 TXS0108ERGYRGY, IC4 TXS0108ERGYRGY, IC5 PTR08100W, IC6 AP1115

Commit message: OE is now tied to 3V3!!!! <--- this enables the logic level..
Connections:
- net 3V3: now also IC2.10, IC3.10, IC4.10
- net GND: no longer IC2.10, IC3.10, IC4.10
Routing:
- net 3V3: track 50.2 -> 67.3 mm, vias 9 -> 12
- net TWCK: track 28.3 -> 24.3 mm
Changed lines of the file:
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@@
 <vertex x="2.794" y="-5.842"/>
 </polygon>
-<contactref element="IC4" pad="10"/>
-<contactref element="IC3" pad="10"/>
-<contactref element="IC2" pad="10"/>
 </signal>
 <signal name="VREF">
@@
 <wire x1="4.572" y1="0.254" x2="5.08" y2="0.762" width="0.254" layer="16"/>
 <wire x1="4.572" y1="-1.016" x2="4.572" y2="0.254" width="0.254" layer="16"/>
-<wire x1="8.636" y1="-5.08" x2="4.572" y2="-1.016" width="0.254" layer="16"/>
-<wire x1="8.636" y1="-7.112" x2="8.636" y2="-5.08" width="0.254" layer="16"/>
-<wire x1="8.128" y1="-7.62" x2="8.636" y2="-7.112" width="0.254" layer="16"/>
-<wire x1="8.128" y1="-7.62" x2="-7.62" y2="-7.62" width="0.254" layer="16"/>
 <via x="5.08" y="0.762" extent="1-16" drill="0.3556"/>
+<wire x1="4.572" y1="-1.016" x2="4.5974" y2="-1.016" width="0.254" layer="16"/>
+<wire x1="4.5974" y1="-1.016" x2="7.1374" y2="-3.556" width="0.254" layer="16"/>
+<wire x1="7.1374" y1="-3.556" x2="7.1374" y2="-3.7846" width="0.254" layer="16"/>
+<wire x1="7.1374" y1="-3.7846" x2="3.302" y2="-7.62" width="0.254" layer="16"/>
+<wire x1="3.302" y1="-7.62" x2="-7.62" y2="-7.62" width="0.254" layer="16"/>
 </signal>
 <signal name="MOSI/TX">
@@
 <vertex x="-5.842" y="0.508"/>
 </polygon>
+<contactref element="IC4" pad="10"/>
+<contactref element="IC3" pad="10"/>
+<contactref element="IC2" pad="10"/>
+<wire x1="6.604" y1="4.2926" x2="6.604" y2="3.048" width="0.2032" layer="16"/>
+<via x="4.318" y="7.366" extent="1-16" drill="0.3556"/>
+<wire x1="7.78685625" y1="-7.55718125" x2="7.2160375" y2="-8.128" width="0.2032" layer="1"/>
+<wire x1="7.2160375" y1="-8.128" x2="6.35" y2="-8.128" width="0.2032" layer="1"/>
+<wire x1="6.35" y1="-8.128" x2="6.096" y2="-7.874" width="0.2032" layer="1"/>
+<wire x1="6.096" y1="-7.874" x2="6.096" y2="-6.604" width="0.2032" layer="1"/>
+<via x="6.096" y="-6.604" extent="1-16" drill="0.3556"/>
+<wire x1="-4.765" y1="-7.251" x2="-5.588" y2="-7.251" width="0.2032" layer="1"/>
+<wire x1="-5.588" y1="-7.251" x2="-5.588" y2="-1.778" width="0.2032" layer="1"/>
+<wire x1="-5.588" y1="-1.778" x2="-4.572" y2="-0.762" width="0.2032" layer="1"/>
+<via x="-4.572" y="-0.762" extent="1-16" drill="0.3556"/>
+<wire x1="-0.315" y1="7.759" x2="3.925" y2="7.759" width="0.2032" layer="1"/>
+<wire x1="3.925" y1="7.759" x2="4.318" y2="7.366" width="0.2032" layer="1"/>
 </signal>
 <signal name="PA19">
