File: NSL_LED_Ball/24x16_RGB.sch (EAGLE design)
At the start: 90 parts, among them IC1 TLC5947XLP, IC2 TLC5947XLP, IC3 TLC5947XLP, IC4 MEGA8-AI, IC5 MCP73123, IC6 BLUETOOTH-RN41", IC7 MMA7455L, IC8 OPA344, X1 16Mhz

Commit message: 
Parts:
- removed F1: 1206L150/12SLYR, SparkFun:PTCSMD
- LED1, LED10, LED11, LED12, LED13, LED14, LED15, LED16, LED17, LED18, LED19, LED2, LED20, LED21, LED22, LED23, LED24, LED3, LED4, LED5, LED6, LED7, LED8, LED9: device 16x16_RGB:GM1WA55311A5MM_RGB_EDGE -> 24x16_RGB:GM1WA55311A5MM_RGB_EDGE
Connections:
- removed net VBAT: BATTERY.2, C7.+, F1.1, IC5.VBAT@1, IC5.VBAT@2
- net VCC: now also BATTERY.2, C7.+, IC5.VBAT@1, IC5.VBAT@2; no longer F1.2
Changed lines of the file:
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@@
 <part name="C15" library="slice_noshift" deviceset="CAP" device="0805" value=".1uF"/>
 <part name="GND14" library="SparkFun" deviceset="GND" device=""/>
-<part name="LED1" library="16x16_RGB" deviceset="GM1WA55311A" device="5MM_RGB_EDGE"/>
-<part name="LED2" library="16x16_RGB" deviceset="GM1WA55311A" device="5MM_RGB_EDGE"/>
-<part name="LED3" library="16x16_RGB" deviceset="GM1WA55311A" device="5MM_RGB_EDGE"/>
-<part name="LED4" library="16x16_RGB" deviceset="GM1WA55311A" device="5MM_RGB_EDGE"/>
-<part name="LED5" library="16x16_RGB" deviceset="GM1WA55311A" device="5MM_RGB_EDGE"/>
-<part name="LED6" library="16x16_RGB" deviceset="GM1WA55311A" device="5MM_RGB_EDGE"/>
-<part name="LED7" library="16x16_RGB" deviceset="GM1WA55311A" device="5MM_RGB_EDGE"/>
-<part name="LED8" library="16x16_RGB" deviceset="GM1WA55311A" device="5MM_RGB_EDGE"/>
-<part name="LED9" library="16x16_RGB" deviceset="GM1WA55311A" device="5MM_RGB_EDGE"/>
-<part name="LED10" library="16x16_RGB" deviceset="GM1WA55311A" device="5MM_RGB_EDGE"/>
-<part name="LED11" library="16x16_RGB" deviceset="GM1WA55311A" device="5MM_RGB_EDGE"/>
-<part name="LED12" library="16x16_RGB" deviceset="GM1WA55311A" device="5MM_RGB_EDGE"/>
-<part name="LED13" library="16x16_RGB" deviceset="GM1WA55311A" device="5MM_RGB_EDGE"/>
-<part name="LED14" library="16x16_RGB" deviceset="GM1WA55311A" device="5MM_RGB_EDGE"/>
-<part name="LED15" library="16x16_RGB" deviceset="GM1WA55311A" device="5MM_RGB_EDGE"/>
-<part name="LED16" library="16x16_RGB" deviceset="GM1WA55311A" device="5MM_RGB_EDGE"/>
-<part name="LED17" library="16x16_RGB" deviceset="GM1WA55311A" device="5MM_RGB_EDGE"/>
-<part name="LED18" library="16x16_RGB" deviceset="GM1WA55311A" device="5MM_RGB_EDGE"/>
-<part name="LED19" library="16x16_RGB" deviceset="GM1WA55311A" device="5MM_RGB_EDGE"/>
-<part name="LED20" library="16x16_RGB" deviceset="GM1WA55311A" device="5MM_RGB_EDGE"/>
-<part name="LED21" library="16x16_RGB" deviceset="GM1WA55311A" device="5MM_RGB_EDGE"/>
-<part name="LED22" library="16x16_RGB" deviceset="GM1WA55311A" device="5MM_RGB_EDGE"/>
-<part name="LED23" library="16x16_RGB" deviceset="GM1WA55311A" device="5MM_RGB_EDGE"/>
-<part name="LED24" library="16x16_RGB" deviceset="GM1WA55311A" device="5MM_RGB_EDGE"/>
+<part name="LED1" library="24x16_RGB" deviceset="GM1WA55311A" device="5MM_RGB_EDGE"/>
+<part name="LED2" library="24x16_RGB" deviceset="GM1WA55311A" device="5MM_RGB_EDGE"/>
+<part name="LED3" library="24x16_RGB" deviceset="GM1WA55311A" device="5MM_RGB_EDGE"/>
+<part name="LED4" library="24x16_RGB" deviceset="GM1WA55311A" device="5MM_RGB_EDGE"/>
+<part name="LED5" library="24x16_RGB" deviceset="GM1WA55311A" device="5MM_RGB_EDGE"/>
+<part name="LED6" library="24x16_RGB" deviceset="GM1WA55311A" device="5MM_RGB_EDGE"/>
+<part name="LED7" library="24x16_RGB" deviceset="GM1WA55311A" device="5MM_RGB_EDGE"/>
+<part name="LED8" library="24x16_RGB" deviceset="GM1WA55311A" device="5MM_RGB_EDGE"/>
+<part name="LED9" library="24x16_RGB" deviceset="GM1WA55311A" device="5MM_RGB_EDGE"/>
+<part name="LED10" library="24x16_RGB" deviceset="GM1WA55311A" device="5MM_RGB_EDGE"/>
+<part name="LED11" library="24x16_RGB" deviceset="GM1WA55311A" device="5MM_RGB_EDGE"/>
+<part name="LED12" library="24x16_RGB" deviceset="GM1WA55311A" device="5MM_RGB_EDGE"/>
+<part name="LED13" library="24x16_RGB" deviceset="GM1WA55311A" device="5MM_RGB_EDGE"/>
+<part name="LED14" library="24x16_RGB" deviceset="GM1WA55311A" device="5MM_RGB_EDGE"/>
+<part name="LED15" library="24x16_RGB" deviceset="GM1WA55311A" device="5MM_RGB_EDGE"/>
+<part name="LED16" library="24x16_RGB" deviceset="GM1WA55311A" device="5MM_RGB_EDGE"/>
+<part name="LED17" library="24x16_RGB" deviceset="GM1WA55311A" device="5MM_RGB_EDGE"/>
+<part name="LED18" library="24x16_RGB" deviceset="GM1WA55311A" device="5MM_RGB_EDGE"/>
+<part name="LED19" library="24x16_RGB" deviceset="GM1WA55311A" device="5MM_RGB_EDGE"/>
+<part name="LED20" library="24x16_RGB" deviceset="GM1WA55311A" device="5MM_RGB_EDGE"/>
+<part name="LED21" library="24x16_RGB" deviceset="GM1WA55311A" device="5MM_RGB_EDGE"/>
+<part name="LED22" library="24x16_RGB" deviceset="GM1WA55311A" device="5MM_RGB_EDGE"/>
+<part name="LED23" library="24x16_RGB" deviceset="GM1WA55311A" device="5MM_RGB_EDGE"/>
+<part name="LED24" library="24x16_RGB" deviceset="GM1WA55311A" device="5MM_RGB_EDGE"/>
 <part name="BATTERY" library="SparkFun" deviceset="M02" device="PTH"/>
 <part name="GND2" library="SparkFun" deviceset="GND" device=""/>
@@
 <part name="GND8" library="SparkFun" deviceset="GND" device=""/>
 <part name="R4" library="slice_noshift" deviceset="RESISTOR" device="0805" value="1K"/>
-<part name="F1" library="SparkFun" deviceset="PTC" device="SMD" value="1206L150/12SLYR"/>
 <part name="C16" library="slice_noshift" deviceset="CAP_POL" device="3528" value="4.7uF"/>
 <part name="GND15" library="SparkFun" deviceset="GND" device=""/>
@@
 <instance part="GND8" gate="1" x="33.02" y="-20.32"/>
 <instance part="R4" gate="G$1" x="-30.48" y="-7.62" rot="R90"/>
-<instance part="F1" gate="G$1" x="83.82" y="0"/>
 <instance part="C16" gate="G$1" x="114.3" y="-2.54"/>
 <instance part="GND15" gate="1" x="114.3" y="-12.7"/>
@@
 </busses>
 <nets>
-<net name="VBAT" class="0">
-<segment>
-<wire x1="68.58" y1="0" x2="78.74" y2="0" width="0.1524" layer="91"/>
-<wire x1="20.32" y1="7.62" x2="27.94" y2="7.62" width="0.1524" layer="91"/>
-<wire x1="27.94" y1="7.62" x2="43.18" y2="7.62" width="0.1524" layer="91"/>
-<wire x1="20.32" y1="2.54" x2="27.94" y2="2.54" width="0.1524" layer="91"/>
-<wire x1="27.94" y1="2.54" x2="27.94" y2="7.62" width="0.1524" layer="91"/>
-<wire x1="43.18" y1="5.08" x2="43.18" y2="7.62" width="0.1524" layer="91"/>
-<wire x1="43.18" y1="7.62" x2="68.58" y2="7.62" width="0.1524" layer="91"/>
-<wire x1="68.58" y1="7.62" x2="68.58" y2="0" width="0.1524" layer="91"/>
-<junction x="27.94" y="7.62"/>
-<junction x="68.58" y="0"/>
-<junction x="43.18" y="7.62"/>
-<pinref part="BATTERY" gate="G$1" pin="2"/>
-<pinref part="IC5" gate="G$1" pin="VBAT@1"/>
-<pinref part="IC5" gate="G$1" pin="VBAT@2"/>
-<pinref part="C7" gate="G$1" pin="+"/>
-<pinref part="F1" gate="G$1" pin="1"/>
-</segment>
-</net>
 <net name="GND" class="0">
 <segment>
@@
 <net name="VCC" class="0">
 <segment>
-<wire x1="91.44" y1="0" x2="114.3" y2="0" width="0.1524" layer="91"/>
 <label x="101.6" y="0" size="1.778" layer="95"/>
-<pinref part="F1" gate="G$1" pin="2"/>
 <pinref part="C16" gate="G$1" pin="+"/>
-</segment>
-</net>
+<wire x1="20.32" y1="7.62" x2="27.94" y2="7.62" width="0.1524" layer="91"/>
+<wire x1="27.94" y1="7.62" x2="43.18" y2="7.62" width="0.1524" layer="91"/>
+<wire x1="20.32" y1="2.54" x2="27.94" y2="2.54" width="0.1524" layer="91"/>
+<wire x1="27.94" y1="2.54" x2="27.94" y2="7.62" width="0.1524" layer="91"/>
+<wire x1="43.18" y1="5.08" x2="43.18" y2="7.62" width="0.1524" layer="91"/>
+<wire x1="43.18" y1="7.62" x2="68.58" y2="7.62" width="0.1524" layer="91"/>
+<wire x1="68.58" y1="7.62" x2="68.58" y2="0" width="0.1524" layer="91"/>
+<junction x="27.94" y="7.62"/>
+<junction x="68.58" y="0"/>
+<junction x="43.18" y="7.62"/>
+<pinref part="BATTERY" gate="G$1" pin="2"/>
+<pinref part="IC5" gate="G$1" pin="VBAT@1"/>
+<pinref part="IC5" gate="G$1" pin="VBAT@2"/>
+<pinref part="C7" gate="G$1" pin="+"/>
+<wire x1="114.3" y1="0" x2="68.58" y2="0" width="0.1524" layer="91"/>
+</segment>
+</net>

Commit message: 
Parts:
- added BATTERY1: (no value), SparkFun:M02PTH
- added Q2: BSH201, transistor-small-signal:BSS84
- added R16: 220K, slice_noshift:RESISTOR0805
- added R17, R18: 10k, SparkFun:RESISTOR
- added R19: 0ohm DNP, SparkFun:RESISTOR
Connections:
- new net BT_PWR: IC4.PD2(INT0), R18.2
- new net N$18: Q2.G, R17.1, R18.1
- new net VDD: C8.1, IC6.VDD, LED.A, Q2.D, R19.1, R6.2, R7.2, R8.2, R9.2
- net BATTSENSE: now also R16.2
- net GND: now also BATTERY1.1
- net VCC: now also BATTERY1.2, Q2.S, R16.1, R17.2, R19.2; no longer C8.1, IC6.VDD, LED.A, R6.2, R7.2, R8.2, R9.2
