File: TV_Nullifier/TV_b_Null_LiPo/tvbgone-2layer.sch (EAGLE design)
At the start: 17 parts, among them IC1 ATTINY85V-10S, Q1 BC857AT115, Q2 FMB2222A, Y1_8MHZ RESONATOR

Commit message: 
Parts:
- removed S1: SWITCH, SparkFun:SWITCH-MOMENTARY-2SMD
- added S2: (no value), SparkFun-Electromechanical:SWITCH-SPDT-SMD-A
- added S3: SWITCH-MOMENTARY-2-SMD-1101NE, SparkFun-Electromechanical:SWITCH-MOMENTARY-2-SMD-1101NE
- C3: value 100uF -> (none); device SparkFun:CAP_POL7343 -> tvbgone-2layer:SPARKFUN_CAP_POL3528
- LED3: device minimidi:LEDCHIPLED_1206 -> minimidi:LEDCHIPLED_0603
- Q2: value FMB2222A -> PMBT3904VS_DUAL_NPN; device fairchild-semic:DUALNPN -> tvbgone-2layer:PMBT3904VS_DUAL_NPN
- R1: device SparkFun:RESISTOR1206 -> SparkFun:RESISTOR
Connections:
- removed net N$7: Q1.C, Q2G$1.B, Q2G$2.B, R3.1
- new net N$8: BAT1.+, S2.O
- new net N$9: Q1.C, Q2A.B, Q2B.B, R3.1
- net GND: now also Q2A.E, Q2B.E, S3.1; no longer Q2G$1.E, Q2G$2.E, S1.2, S1.3
- net N$4: now also Q2A.C; no longer Q2G$2.C
- net N$5: now also Q2B.C; no longer Q2G$1.C
- net RST: now also S3.2; no longer S1.4
- net VCC: now also S2.P; no longer BAT1.+
Other:
- moved on the sheet: C3
