File: NSL_RGB_LED_Ball/24x16_RGB_Top.sch (EAGLE design)
At the start: 16 parts

Commit message: 
Parts:
- added JP2: (no value), SparkFun-Connectors:M06SIP
- added S1, S2: SPARKFUN-ELECTROMECHANICAL_SWITCH-MOMENTARY-2-SMD-1101NE, tvbgone-2layer:SPARKFUN-ELECTROMECHANICAL_SWITCH-MOMENTARY-2-SMD-1101NE
- added U$1: USB_PANNEL, 24x16_RGB_Bottom:USB_PANNEL
- SLOT1, SLOT10, SLOT11, SLOT12, SLOT13, SLOT14, SLOT15, SLOT16, SLOT2, SLOT3, SLOT4, SLOT5, SLOT6, SLOT7, SLOT8, SLOT9: device slice:SLOT -> 24x16_RGB_Bottom:SLOT
Connections:
- new net MODE: JP2.4, JP2.6, S1.1
- new net RST: JP2.1, JP2.3, S2.1
- net BLANK: now also SLOT1.P$1, SLOT1.P$2, SLOT10.P$1, SLOT10.P$2, SLOT11.P$1, SLOT11.P$2, SLOT12.P$1, SLOT12.P$2, SLOT13.P$1, SLOT13.P$2, SLOT14.P$1, SLOT14.P$2, SLOT15.P$1, SLOT15.P$2, SLOT16.P$1, SLOT16.P$2, SLOT2.P$1, SLOT2.P$2, SLOT3.P$1, SLOT3.P$2, SLOT4.P$1, SLOT4.P$2, SLOT5.P$1, SLOT5.P$2, SLOT6.P$1, SLOT6.P$2, SLOT7.P$1, SLOT7.P$2, SLOT8.P$1, SLOT8.P$2, SLOT9.P$1, SLOT9.P$2; no longer SLOT1.P$3, SLOT1.P$4, SLOT10.P$3, SLOT10.P$4, SLOT11.P$3, SLOT11.P$4, SLOT12.P$3, SLOT12.P$4, SLOT13.P$3, SLOT13.P$4, SLOT14.P$3, SLOT14.P$4, SLOT15.P$3, SLOT15.P$4, SLOT16.P$3, SLOT16.P$4, SLOT2.P$3, SLOT2.P$4, SLOT3.P$3, SLOT3.P$4, SLOT4.P$3, SLOT4.P$4, SLOT5.P$3, SLOT5.P$4, SLOT6.P$3, SLOT6.P$4, SLOT7.P$3, SLOT7.P$4, SLOT8.P$3, SLOT8.P$4, SLOT9.P$3, SLOT9.P$4
- net GND: now also JP2.2, JP2.5, S1.2, S2.2, SLOT1.P$3, SLOT1.P$4, SLOT10.P$3, SLOT10.P$4, SLOT11.P$3, SLOT11.P$4, SLOT12.P$3, SLOT12.P$4, SLOT13.P$3, SLOT13.P$4, SLOT14.P$3, SLOT14.P$4, SLOT15.P$3, SLOT15.P$4, SLOT16.P$3, SLOT16.P$4, SLOT2.P$3, SLOT2.P$4, SLOT3.P$3, SLOT3.P$4, SLOT4.P$3, SLOT4.P$4, SLOT5.P$3, SLOT5.P$4, SLOT6.P$3, SLOT6.P$4, SLOT7.P$3, SLOT7.P$4, SLOT8.P$3, SLOT8.P$4, SLOT9.P$3, SLOT9.P$4; no longer SLOT1.P$1, SLOT1.P$2, SLOT10.P$1, SLOT10.P$2, SLOT11.P$1, SLOT11.P$2, SLOT12.P$1, SLOT12.P$2, SLOT13.P$1, SLOT13.P$2, SLOT14.P$1, SLOT14.P$2, SLOT15.P$1, SLOT15.P$2, SLOT16.P$1, SLOT16.P$2, SLOT2.P$1, SLOT2.P$2, SLOT3.P$1, SLOT3.P$2, SLOT4.P$1, SLOT4.P$2, SLOT5.P$1, SLOT5.P$2, SLOT6.P$1, SLOT6.P$2, SLOT7.P$1, SLOT7.P$2, SLOT8.P$1, SLOT8.P$2, SLOT9.P$1, SLOT9.P$2
Changed lines of the file:
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@@
 </classes>
 <parts>
-<part name="SLOT1" library="slice" deviceset="SLOT" device="">
-<attribute name="MF" value=""/>
-<attribute name="MPN" value=""/>
-<attribute name="OC_NEWARK" value="unknown"/>
-</part>
-<part name="SLOT2" library="slice" deviceset="SLOT" device="">
-<attribute name="MF" value=""/>
-<attribute name="MPN" value=""/>
-<attribute name="OC_NEWARK" value="unknown"/>
-</part>
-<part name="SLOT3" library="slice" deviceset="SLOT" device="">
-<attribute name="MF" value=""/>
-<attribute name="MPN" value=""/>
-<attribute name="OC_NEWARK" value="unknown"/>
-</part>
-<part name="SLOT4" library="slice" deviceset="SLOT" device="">
-<attribute name="MF" value=""/>
-<attribute name="MPN" value=""/>
-<attribute name="OC_NEWARK" value="unknown"/>
-</part>
-<part name="SLOT5" library="slice" deviceset="SLOT" device="">
-<attribute name="MF" value=""/>
-<attribute name="MPN" value=""/>
-<attribute name="OC_NEWARK" value="unknown"/>
-</part>
-<part name="SLOT6" library="slice" deviceset="SLOT" device="">
-<attribute name="MF" value=""/>
-<attribute name="MPN" value=""/>
-<attribute name="OC_NEWARK" value="unknown"/>
-</part>
-<part name="SLOT7" library="slice" deviceset="SLOT" device="">
-<attribute name="MF" value=""/>
-<attribute name="MPN" value=""/>
-<attribute name="OC_NEWARK" value="unknown"/>
-</part>
-<part name="SLOT8" library="slice" deviceset="SLOT" device="">
-<attribute name="MF" value=""/>
-<attribute name="MPN" value=""/>
-<attribute name="OC_NEWARK" value="unknown"/>
-</part>
-<part name="SLOT9" library="slice" deviceset="SLOT" device="">
-<attribute name="MF" value=""/>
-<attribute name="MPN" value=""/>
-<attribute name="OC_NEWARK" value="unknown"/>
-</part>
-<part name="SLOT10" library="slice" deviceset="SLOT" device="">
-<attribute name="MF" value=""/>
-<attribute name="MPN" value=""/>
-<attribute name="OC_NEWARK" value="unknown"/>
-</part>
-<part name="SLOT11" library="slice" deviceset="SLOT" device="">
-<attribute name="MF" value=""/>
-<attribute name="MPN" value=""/>
-<attribute name="OC_NEWARK" value="unknown"/>
-</part>
-<part name="SLOT12" library="slice" deviceset="SLOT" device="">
-<attribute name="MF" value=""/>
-<attribute name="MPN" value=""/>
-<attribute name="OC_NEWARK" value="unknown"/>
-</part>
-<part name="SLOT13" library="slice" deviceset="SLOT" device="">
-<attribute name="MF" value=""/>
-<attribute name="MPN" value=""/>
-<attribute name="OC_NEWARK" value="unknown"/>
-</part>
-<part name="SLOT14" library="slice" deviceset="SLOT" device="">
-<attribute name="MF" value=""/>
-<attribute name="MPN" value=""/>
-<attribute name="OC_NEWARK" value="unknown"/>
-</part>
-<part name="SLOT15" library="slice" deviceset="SLOT" device="">
-<attribute name="MF" value=""/>
-<attribute name="MPN" value=""/>
-<attribute name="OC_NEWARK" value="unknown"/>
-</part>
-<part name="SLOT16" library="slice" deviceset="SLOT" device="">
-<attribute name="MF" value=""/>
-<attribute name="MPN" value=""/>
-<attribute name="OC_NEWARK" value="unknown"/>
-</part>
+<part name="SLOT1" library="24x16_RGB_Bottom" deviceset="SLOT" device="">
+<attribute name="MF" value=""/>
+<attribute name="MPN" value=""/>
+<attribute name="OC_NEWARK" value="unknown"/>
+</part>
+<part name="SLOT2" library="24x16_RGB_Bottom" deviceset="SLOT" device="">
+<attribute name="MF" value=""/>
+<attribute name="MPN" value=""/>
+<attribute name="OC_NEWARK" value="unknown"/>
+</part>
+<part name="SLOT3" library="24x16_RGB_Bottom" deviceset="SLOT" device="">
+<attribute name="MF" value=""/>
+<attribute name="MPN" value=""/>
+<attribute name="OC_NEWARK" value="unknown"/>
+</part>
+<part name="SLOT4" library="24x16_RGB_Bottom" deviceset="SLOT" device="">
+<attribute name="MF" value=""/>
+<attribute name="MPN" value=""/>
+<attribute name="OC_NEWARK" value="unknown"/>
+</part>
+<part name="SLOT5" library="24x16_RGB_Bottom" deviceset="SLOT" device="">
+<attribute name="MF" value=""/>
+<attribute name="MPN" value=""/>
+<attribute name="OC_NEWARK" value="unknown"/>
+</part>
+<part name="SLOT6" library="24x16_RGB_Bottom" deviceset="SLOT" device="">
+<attribute name="MF" value=""/>
+<attribute name="MPN" value=""/>
+<attribute name="OC_NEWARK" value="unknown"/>
+</part>
+<part name="SLOT7" library="24x16_RGB_Bottom" deviceset="SLOT" device="">
+<attribute name="MF" value=""/>
+<attribute name="MPN" value=""/>
+<attribute name="OC_NEWARK" value="unknown"/>
+</part>
+<part name="SLOT8" library="24x16_RGB_Bottom" deviceset="SLOT" device="">
+<attribute name="MF" value=""/>
+<attribute name="MPN" value=""/>
+<attribute name="OC_NEWARK" value="unknown"/>
+</part>
+<part name="SLOT9" library="24x16_RGB_Bottom" deviceset="SLOT" device="">
+<attribute name="MF" value=""/>
+<attribute name="MPN" value=""/>
+<attribute name="OC_NEWARK" value="unknown"/>
+</part>
+<part name="SLOT10" library="24x16_RGB_Bottom" deviceset="SLOT" device="">
+<attribute name="MF" value=""/>
+<attribute name="MPN" value=""/>
+<attribute name="OC_NEWARK" value="unknown"/>
+</part>
+<part name="SLOT11" library="24x16_RGB_Bottom" deviceset="SLOT" device="">
+<attribute name="MF" value=""/>
+<attribute name="MPN" value=""/>
+<attribute name="OC_NEWARK" value="unknown"/>
+</part>
+<part name="SLOT12" library="24x16_RGB_Bottom" deviceset="SLOT" device="">
+<attribute name="MF" value=""/>
+<attribute name="MPN" value=""/>
+<attribute name="OC_NEWARK" value="unknown"/>
+</part>
+<part name="SLOT13" library="24x16_RGB_Bottom" deviceset="SLOT" device="">
+<attribute name="MF" value=""/>
+<attribute name="MPN" value=""/>
+<attribute name="OC_NEWARK" value="unknown"/>
+</part>
+<part name="SLOT14" library="24x16_RGB_Bottom" deviceset="SLOT" device="">
+<attribute name="MF" value=""/>
+<attribute name="MPN" value=""/>
+<attribute name="OC_NEWARK" value="unknown"/>
+</part>
+<part name="SLOT15" library="24x16_RGB_Bottom" deviceset="SLOT" device="">
+<attribute name="MF" value=""/>
+<attribute name="MPN" value=""/>
+<attribute name="OC_NEWARK" value="unknown"/>
+</part>
+<part name="SLOT16" library="24x16_RGB_Bottom" deviceset="SLOT" device="">
+<attribute name="MF" value=""/>
+<attribute name="MPN" value=""/>
+<attribute name="OC_NEWARK" value="unknown"/>
+</part>
+<part name="S1" library="tvbgone-2layer" deviceset="SPARKFUN-ELECTROMECHANICAL_SWITCH-MOMENTARY-2" device="-SMD-1101NE"/>
+<part name="S2" library="tvbgone-2layer" deviceset="SPARKFUN-ELECTROMECHANICAL_SWITCH-MOMENTARY-2" device="-SMD-1101NE"/>
+<part name="GND1" library="tvbgone-2layer" deviceset="SUPPLY1_GND" device=""/>
+<part name="GND2" library="tvbgone-2layer" deviceset="SUPPLY1_GND" device=""/>
+<part name="JP2" library="SparkFun-Connectors" deviceset="M06" device="SIP"/>
+<part name="U$1" library="24x16_RGB_Bottom" deviceset="USB_PANNEL" device=""/>
 </parts>
 <sheets>
@@
 </busses>
 <nets>
-<net name="BLANK" class="0">
+<net name="GND" class="0">
 <segment>
 <pinref part="SLOT1" gate="G$1" pin="P$3"/>
@@
 </segment>
 </net>
-<net name="GND" class="0">
+<net name="BLANK" class="0">
 <segment>
 <pinref part="SLOT1" gate="G$1" pin="P$1"/>
@@
 </segment>
 </net>
+</nets>
+</sheet>
+<sheet>
+<plain>
+</plain>
+<instances>
+<instance part="S1" gate="G$1" x="55.88" y="81.28"/>
+<instance part="S2" gate="G$1" x="55.88" y="66.04"/>
+<instance part="GND1" gate="1" x="30.48" y="66.04"/>
+<instance part="GND2" gate="1" x="68.58" y="53.34"/>
+<instance part="JP2" gate="G$1" x="0" y="73.66"/>
+<instance part="U$1" gate="G$1" x="68.58" y="40.64"/>
+</instances>
+<busses>
+</busses>
+<nets>
+<net name="MODE" class="0">
+<segment>
+<pinref part="S1" gate="G$1" pin="1"/>
+<wire x1="50.8" y1="81.28" x2="43.18" y2="81.28" width="0.1524" layer="91"/>
+<label x="43.18" y="81.28" size="1.778" layer="95"/>
+</segment>
+<segment>
+<wire x1="5.08" y1="81.28" x2="20.32" y2="81.28" width="0.1524" layer="91"/>
+<label x="12.7" y="81.28" size="1.778" layer="95"/>
+<pinref part="JP2" gate="G$1" pin="6"/>
+</segment>
+<segment>
+<wire x1="5.08" y1="76.2" x2="20.32" y2="76.2" width="0.1524" layer="91"/>
+<pinref part="JP2" gate="G$1" pin="4"/>
+<label x="12.7" y="76.2" size="1.778" layer="95"/>
+</segment>
+</net>
+<net name="RST" class="0">
+<segment>
+<pinref part="S2" gate="G$1" pin="1"/>
+<wire x1="50.8" y1="66.04" x2="43.18" y2="66.04" width="0.1524" layer="91"/>
+<label x="43.18" y="66.04" size="1.778" layer="95"/>
+</segment>
+<segment>
+<wire x1="5.08" y1="68.58" x2="20.32" y2="68.58" width="0.1524" layer="91"/>
+<label x="12.7" y="68.58" size="1.778" layer="95"/>
+<pinref part="JP2" gate="G$1" pin="1"/>
+</segment>
+<segment>
+<wire x1="5.08" y1="73.66" x2="20.32" y2="73.66" width="0.1524" layer="91"/>
+<pinref part="JP2" gate="G$1" pin="3"/>
+<label x="12.7" y="73.66" size="1.778" layer="95"/>
+</segment>
+</net>
+<net name="GND" class="0">
+<segment>
+<wire x1="30.48" y1="76.2" x2="30.48" y2="73.66" width="0.1524" layer="91"/>
+<wire x1="30.48" y1="73.66" x2="30.48" y2="71.12" width="0.1524" layer="91"/>
+<wire x1="30.48" y1="71.12" x2="30.48" y2="68.58" width="0.1524" layer="91"/>
+<pinref part="GND1" gate="1" pin="GND"/>
+<pinref part="JP2" gate="G$1" pin="5"/>
+<wire x1="5.08" y1="78.74" x2="30.48" y2="78.74" width="0.1524" layer="91"/>
+<wire x1="30.48" y1="78.74" x2="30.48" y2="76.2" width="0.1524" layer="91"/>
+<pinref part="JP2" gate="G$1" pin="2"/>
+<wire x1="5.08" y1="71.12" x2="30.48" y2="71.12" width="0.1524" layer="91"/>
+</segment>
+<segment>
+<pinref part="S1" gate="G$1" pin="2"/>
+<wire x1="60.96" y1="81.28" x2="68.58" y2="81.28" width="0.1524" layer="91"/>
+<wire x1="68.58" y1="81.28" x2="68.58" y2="66.04" width="0.1524" layer="91"/>
+<pinref part="S2" gate="G$1" pin="2"/>
+<wire x1="68.58" y1="66.04" x2="68.58" y2="55.88" width="0.1524" layer="91"/>
+<wire x1="60.96" y1="66.04" x2="68.58" y2="66.04" width="0.1524" layer="91"/>
+<junction x="68.58" y="66.04"/>
+<pinref part="GND2" gate="1" pin="GND"/>
+</segment>
+</net>
