File: Motor Control/yoocnc_grbl/yoocnc_grbl.sch (EAGLE design)
At the start: 121 parts, among them IC1 A4983, IC2 LM317L, IC3 FT232RL, IC4 A4983, IC5 ATMEGA2560AU, IC6 A4983, Q2 16MHz

Commit message: ERC fixed.
Parts:
- renumbered Q2 to Q1
Connections:
- net N$56: no longer Q1.1
- net N$57: no longer Q1.2
Changed lines of the file:
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@@
 <?xml version="1.0" encoding="utf-8"?>
 <!DOCTYPE eagle SYSTEM "eagle.dtd">
-<eagle version="6.4">
+<eagle version="6.5.0">
 <drawing>
 <settings>
@@
 <part name="GND13" library="supply1" deviceset="GND" device=""/>
 <part name="GND21" library="supply1" deviceset="GND" device=""/>
-<part name="Q2" library="crystal" deviceset="CRYTAL" device="SM49" value="16MHz">
-<attribute name="PARTNO" value="ABLS-16.000MHZ-B4-T"/>
-</part>
 <part name="C26" library="resistor" deviceset="C-EU" device="C0805K" value="100n">
 <attribute name="PARTNO" value="CC0805ZRY5V9BB104"/>
@@
 <part name="R61" library="resistor" deviceset="R-EU_" device="R0603" value="20K">
 <attribute name="PARTNO" value="RC0805JR-0710KL"/>
+</part>
+<part name="Q1" library="crystal" deviceset="CRYTAL" device="SM49" value="16MHz">
+<attribute name="PARTNO" value="ABLS-16.000MHZ-B4-T"/>
 </part>
 </parts>
@@
 <attribute name="VALUE" x="-33.655" y="117.475" size="1.778" layer="96"/>
 </instance>
-<instance part="Q2" gate="G$1" x="-16.51" y="117.475" smashed="yes" rot="R90">
-<attribute name="NAME" x="-10.16" y="121.539" size="1.778" layer="95" rot="R180"/>
-<attribute name="VALUE" x="-13.335" y="116.84" size="1.778" layer="96"/>
-<attribute name="PARTNO" x="-16.51" y="117.475" size="1.778" layer="96" display="off"/>
-</instance>
 <instance part="C26" gate="G$1" x="-43.18" y="97.79" smashed="yes" rot="MR0">
 <attribute name="NAME" x="-44.704" y="98.171" size="1.778" layer="95" rot="MR0"/>
@@
 <attribute name="VALUE" x="116.84" y="-16.002" size="1.778" layer="96"/>
 <attribute name="PARTNO" x="119.38" y="-12.7" size="1.778" layer="96" rot="R270" display="off"/>
+</instance>
+<instance part="Q1" gate="G$1" x="-16.51" y="117.475" smashed="yes" rot="R90">
+<attribute name="NAME" x="-10.16" y="121.539" size="1.778" layer="95" rot="R180"/>
+<attribute name="VALUE" x="-13.335" y="116.84" size="1.778" layer="96"/>
+<attribute name="PARTNO" x="-16.51" y="117.475" size="1.778" layer="96" display="off"/>
 </instance>
 </instances>
@@
 <wire x1="-16.51" y1="114.935" x2="-16.51" y2="112.395" width="0.1524" layer="91"/>
 <junction x="-16.51" y="112.395"/>
-<pinref part="Q2" gate="G$1" pin="1"/>
 <pinref part="C28" gate="G$1" pin="2"/>
 <pinref part="IC5" gate="1" pin="XTAL1"/>
@@
 <wire x1="-16.51" y1="120.015" x2="-16.51" y2="122.555" width="0.1524" layer="91"/>
 <junction x="-16.51" y="122.555"/>
-<pinref part="Q2" gate="G$1" pin="2"/>
 <pinref part="C29" gate="G$1" pin="2"/>
 <pinref part="IC5" gate="1" pin="XTAL2"/>
