File: Motor Control/yoocnc_grbl/yoocnc_grbl.brd (EAGLE design)
At the start: 99.8 x 80 mm, 121 parts, among them IC1 A4983, IC2 LM317L, IC3 FT232RL, IC4 A4983, IC5 ATMEGA2560AU, IC6 A4983, Q2 16MHz

Commit message: ERC fixed.
Parts:
- removed Q2: 16MHz, crystal:SM49@1
- added Q1: 16MHz, crystal:SM49
- moved 3/5V 2.54 mm to (98.7, 95.2)
- moved R36 2.29 mm to (112.3, 74.6)
- moved C30 1.68 mm to (87.6, 72.1)
- moved C2 1.27 mm to (100.3, 92.8)
- moved R45 1.27 mm to (95.4, 37.5)
- moved R6 1.27 mm to (102.8, 94.8)
- moved R7 1.27 mm to (100.8, 95.3)
- moved C13 0.24 mm to (122.5, 57.2)
- moved R13 0.22 mm to (115.6, 76.4)
- moved C23 0.16 mm to (122.5, 41.5)
- moved C22 0.12 mm to (122.6, 36.1)
- moved C1 0.08 mm to (108.2, 91.4)
Connections:
- net N$56: no longer Q2.1
- net N$57: no longer Q2.2
Routing:
- net Z_COILB-: track 22.5 -> 45.6 mm
- net X_COILA+: track 27.5 -> 48.2 mm
- net Z_COILA-: track 35.4 -> 54.2 mm
- net X_COILB-: track 28.8 -> 46.1 mm
- net V+: track 128.3 -> 144.6 mm, vias 11 -> 15
- net Z_COILB+: track 29.2 -> 44.4 mm
- net Y_COILA+: track 32.0 -> 46.5 mm
- net Y_COILB-: track 28.2 -> 39.6 mm
- net Y_COILB+: track 29.4 -> 40.6 mm
- net Z_COILA+: track 36.5 -> 46.6 mm
- net Y_COILA-: track 20.8 -> 30.6 mm
- net YL2: track 27.5 -> 35.9 mm
- net XL1: track 30.1 -> 38.0 mm
- net ZL1: track 27.8 -> 35.5 mm
- net X_COILA-: track 22.7 -> 29.9 mm
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Other:
- board text added: "[NSL] http://www.nullspacelabs.com"

Commit message: fixes
Routing:
- net GND: track 43.4 -> 47.7 mm
- net V+: track 144.6 -> 146.6 mm
- net ENABLE: track 111.1 -> 112.0 mm
- net USBVCC: track 254.8 -> 255.4 mm
Changed lines of the file:
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@@
 <via x="120.65" y="50.8" extent="1-16" drill="0.6096"/>
 <via x="120.65" y="49.53" extent="1-16" drill="0.6096"/>
-<via x="120.65" y="48.26" extent="1-16" drill="0.6096"/>
+<via x="119.38" y="49.53" extent="1-16" drill="0.6096"/>
 <via x="119.38" y="48.26" extent="1-16" drill="0.6096"/>
 <via x="118.11" y="48.26" extent="1-16" drill="0.6096"/>
@@
 <wire x1="98.715" y1="95.65" x2="98.993" y2="95.928" width="0.1778" layer="1"/>
 <wire x1="98.993" y1="95.928" x2="100.832" y2="95.928" width="0.508" layer="1"/>
-<wire x1="68.887" y1="80.403" x2="70.837" y2="80.403" width="0" layer="19" extent="1-1"/>
+<wire x1="70.837" y1="80.403" x2="70.837" y2="81.704559375" width="0.1778" layer="1"/>
+<wire x1="70.837" y1="81.704559375" x2="71.014071875" y2="81.88163125" width="0.1778" layer="1" curve="-90"/>
+<wire x1="71.014071875" y1="81.88163125" x2="71.014071875" y2="81.446246875" width="0.1778" layer="1"/>
+<wire x1="71.014071875" y1="81.446246875" x2="70.822946875" y2="81.255121875" width="0.1778" layer="1" curve="-90"/>
+<wire x1="70.822946875" y1="81.255121875" x2="70.822946875" y2="79.364965625" width="0.1778" layer="1"/>
+<wire x1="70.822946875" y1="79.364965625" x2="70.929128125" y2="79.258784375" width="0.1778" layer="1" curve="90"/>
 </signal>
 <signal name="VCC">
@@
 <wire x1="123.825" y1="82.524" x2="123.825" y2="85.09" width="0.1778" layer="1"/>
 <wire x1="123.825" y1="61.6585" x2="123.825" y2="62.9285" width="0.635" layer="1"/>
-<wire x1="114.948" y1="85.852" x2="114.95" y2="85.924" width="0" layer="19" extent="1-1"/>
-<wire x1="115.369490625" y1="85.852" x2="115.57" y2="85.852" width="0" layer="19" extent="1-16"/>
-<wire x1="114.95" y1="43.633" x2="115.1405" y2="43.688" width="0" layer="19" extent="1-1"/>
+<wire x1="115.57" y1="85.852" x2="114.95" y2="85.924" width="0.1778" layer="1"/>
+<wire x1="115.369490625" y1="85.852" x2="115.57" y2="86.36" width="0.1778" layer="16"/>
+<wire x1="115.57" y1="86.36" x2="115.568315625" y2="85.73711875" width="0.1778" layer="16"/>
+<wire x1="115.1405" y1="43.688" x2="114.95" y2="43.633" width="0.1778" layer="1"/>
 </signal>
 <signal name="N$6">
@@
 <wire x1="137.902665625" y1="32.66336875" x2="137.921403125" y2="32.66336875" width="0.1778" layer="1"/>
 <wire x1="137.921403125" y1="32.66336875" x2="138.113440625" y2="32.959475" width="0.1778" layer="1"/>
-<wire x1="120.892884375" y1="36.066115625" x2="120.522" y2="36.378" width="0" layer="19" extent="1-1"/>
+<wire x1="120.892884375" y1="36.066115625" x2="120.522" y2="36.378" width="0.1778" layer="1"/>
 </signal>
 <signal name="Z_STEP">
@@
 <wire x1="94.615" y1="85.778" x2="94.672" y2="85.778" width="0.3048" layer="1"/>
 <wire x1="120.022" y1="46.221" x2="120.015" y2="46.228" width="0.3048" layer="1"/>
-<wire x1="120.0091875" y1="63.21044375" x2="120.022" y2="63.246" width="0.3048" layer="1"/>
-<wire x1="120.022" y1="63.246" x2="120.022" y2="62.178" width="0.3048" layer="1"/>
-<wire x1="115.71515" y1="62.738" x2="120.55216875" y2="62.738" width="0.3048" layer="16"/>
 <wire x1="120.55216875" y1="62.738" x2="121.92" y2="61.37016875" width="0.3048" layer="16" curve="-90"/>
 <wire x1="121.92" y1="61.37016875" x2="121.92" y2="50.944178125" width="0.3048" layer="16"/>
@@
 <wire x1="95.25" y1="85.598" x2="94.996" y2="85.598" width="0.3048" layer="16"/>
 <wire x1="113.883609375" y1="84.2660625" x2="113.883609375" y2="64.628165625" width="0.3048" layer="16"/>
-<wire x1="113.883609375" y1="64.628165625" x2="114.44936875" y2="63.262303125" width="0.3048" layer="16" curve="45.000066"/>
-<wire x1="114.44936875" y1="63.262303125" x2="115.71515" y2="62.738" width="0.3048" layer="16" curve="45"/>
 <wire x1="109.982" y1="84.328" x2="113.883609375" y2="84.2660625" width="0.3048" layer="16"/>
 <wire x1="94.742" y1="85.852" x2="94.742" y2="87.2925" width="0.3048" layer="1"/>
@@
 <wire x1="94.615" y1="85.778" x2="94.615" y2="85.8012" width="0.3048" layer="1"/>
 <wire x1="94.615" y1="85.8012" x2="94.742" y2="85.852" width="0.3048" layer="1"/>
-<via x="120.0091875" y="63.21044375" extent="1-16" drill="0.3556"/>
 <via x="120.022" y="46.221" extent="1-16" drill="0.6096"/>
 <via x="119.8245" y="84.328" extent="1-16" drill="0.3556"/>
 <via x="94.742" y="85.852" extent="1-16" drill="0.6096"/>
-<wire x1="120.55216875" y1="62.738" x2="120.022" y2="63.246" width="0" layer="19" extent="1-16"/>
+<wire x1="120.0091875" y1="62.738" x2="120.55216875" y2="62.738" width="0.3048" layer="16"/>
+<wire x1="115.265775" y1="63.246" x2="113.883609375" y2="64.628165625" width="0.3048" layer="16" curve="-90"/>
+<wire x1="120.022" y1="62.178" x2="120.024275" y2="62.180275" width="0.3048" layer="1" curve="90"/>
+<via x="120.008640625" y="63.213725" extent="1-16" drill="0.3556"/>
+<wire x1="120.008640625" y1="63.213725" x2="120.0091875" y2="63.37641875" width="0.3048" layer="16" curve="90"/>
+<wire x1="120.0091875" y1="63.37641875" x2="120.0091875" y2="62.738" width="0.3048" layer="16"/>
+<wire x1="119.98479375" y1="63.231115625" x2="119.463965625" y2="63.231115625" width="0.3048" layer="16"/>
+<wire x1="119.463965625" y1="63.231115625" x2="115.280659375" y2="63.231115625" width="0.3048" layer="16"/>
+<wire x1="115.280659375" y1="63.231115625" x2="115.265775" y2="63.246" width="0.3048" layer="16" curve="-90"/>
+<wire x1="120.0091875" y1="63.37641875" x2="119.60926875" y2="63.37641875" width="0.3048" layer="16"/>
+<wire x1="119.60926875" y1="63.37641875" x2="119.463965625" y2="63.231115625" width="0.3048" layer="16" curve="90"/>
+<wire x1="120.022" y1="62.178" x2="120.022" y2="63.200365625" width="0.3048" layer="1"/>
+<wire x1="120.022" y1="63.200365625" x2="120.008640625" y2="63.213725" width="0.3048" layer="1" curve="90"/>
 </signal>
 <signal name="SLEEP">
@@
 <wire x1="86.62885" y1="72.0668" x2="86.614" y2="72.08165" width="0.508" layer="1"/>
 <wire x1="86.614" y1="72.08165" x2="86.614" y2="74.27140625" width="0.508" layer="1"/>
-<wire x1="70.187" y1="80.403" x2="69.537" y2="80.403" width="0" layer="19" extent="1-1"/>
+<wire x1="69.537" y1="80.403" x2="70.187" y2="80.403" width="0.508" layer="1"/>
 </signal>
 <signal name="CTS">
