File: NSL_RGB_LED_Ball/Botton/24x16_RGB_Bottom.sch (EAGLE design)
At the start: 20 parts

Commit message: 
Parts:
- SLOT1, SLOT10, SLOT11, SLOT12, SLOT13, SLOT14, SLOT15, SLOT16, SLOT2, SLOT3, SLOT4, SLOT5, SLOT6, SLOT7, SLOT8, SLOT9: device 24x16_RGB_Bottom:SLOT -> 24x16_RGB_Top:SLOT
Changed lines of the file:
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@@
 </classes>
 <parts>
-<part name="SLOT1" library="24x16_RGB_Bottom" deviceset="SLOT" device="">
+<part name="SLOT1" library="24x16_RGB_Top" deviceset="SLOT" device="">
 <attribute name="MF" value=""/>
 <attribute name="MPN" value=""/>
 <attribute name="OC_NEWARK" value="unknown"/>
 </part>
-<part name="SLOT2" library="24x16_RGB_Bottom" deviceset="SLOT" device="">
+<part name="SLOT2" library="24x16_RGB_Top" deviceset="SLOT" device="">
 <attribute name="MF" value=""/>
 <attribute name="MPN" value=""/>
 <attribute name="OC_NEWARK" value="unknown"/>
 </part>
-<part name="SLOT3" library="24x16_RGB_Bottom" deviceset="SLOT" device="">
+<part name="SLOT3" library="24x16_RGB_Top" deviceset="SLOT" device="">
 <attribute name="MF" value=""/>
 <attribute name="MPN" value=""/>
 <attribute name="OC_NEWARK" value="unknown"/>
 </part>
-<part name="SLOT4" library="24x16_RGB_Bottom" deviceset="SLOT" device="">
+<part name="SLOT4" library="24x16_RGB_Top" deviceset="SLOT" device="">
 <attribute name="MF" value=""/>
 <attribute name="MPN" value=""/>
 <attribute name="OC_NEWARK" value="unknown"/>
 </part>
-<part name="SLOT5" library="24x16_RGB_Bottom" deviceset="SLOT" device="">
+<part name="SLOT5" library="24x16_RGB_Top" deviceset="SLOT" device="">
 <attribute name="MF" value=""/>
 <attribute name="MPN" value=""/>
 <attribute name="OC_NEWARK" value="unknown"/>
 </part>
-<part name="SLOT6" library="24x16_RGB_Bottom" deviceset="SLOT" device="">
+<part name="SLOT6" library="24x16_RGB_Top" deviceset="SLOT" device="">
 <attribute name="MF" value=""/>
 <attribute name="MPN" value=""/>
 <attribute name="OC_NEWARK" value="unknown"/>
 </part>
-<part name="SLOT7" library="24x16_RGB_Bottom" deviceset="SLOT" device="">
+<part name="SLOT7" library="24x16_RGB_Top" deviceset="SLOT" device="">
 <attribute name="MF" value=""/>
 <attribute name="MPN" value=""/>
 <attribute name="OC_NEWARK" value="unknown"/>
 </part>
-<part name="SLOT8" library="24x16_RGB_Bottom" deviceset="SLOT" device="">
+<part name="SLOT8" library="24x16_RGB_Top" deviceset="SLOT" device="">
 <attribute name="MF" value=""/>
 <attribute name="MPN" value=""/>
 <attribute name="OC_NEWARK" value="unknown"/>
 </part>
-<part name="SLOT9" library="24x16_RGB_Bottom" deviceset="SLOT" device="">
+<part name="SLOT9" library="24x16_RGB_Top" deviceset="SLOT" device="">
 <attribute name="MF" value=""/>
 <attribute name="MPN" value=""/>
 <attribute name="OC_NEWARK" value="unknown"/>
 </part>
-<part name="SLOT10" library="24x16_RGB_Bottom" deviceset="SLOT" device="">
+<part name="SLOT10" library="24x16_RGB_Top" deviceset="SLOT" device="">
 <attribute name="MF" value=""/>
 <attribute name="MPN" value=""/>
 <attribute name="OC_NEWARK" value="unknown"/>
 </part>
-<part name="SLOT11" library="24x16_RGB_Bottom" deviceset="SLOT" device="">
+<part name="SLOT11" library="24x16_RGB_Top" deviceset="SLOT" device="">
 <attribute name="MF" value=""/>
 <attribute name="MPN" value=""/>
 <attribute name="OC_NEWARK" value="unknown"/>
 </part>
-<part name="SLOT12" library="24x16_RGB_Bottom" deviceset="SLOT" device="">
+<part name="SLOT12" library="24x16_RGB_Top" deviceset="SLOT" device="">
 <attribute name="MF" value=""/>
 <attribute name="MPN" value=""/>
 <attribute name="OC_NEWARK" value="unknown"/>
 </part>
-<part name="SLOT13" library="24x16_RGB_Bottom" deviceset="SLOT" device="">
+<part name="SLOT13" library="24x16_RGB_Top" deviceset="SLOT" device="">
 <attribute name="MF" value=""/>
 <attribute name="MPN" value=""/>
 <attribute name="OC_NEWARK" value="unknown"/>
 </part>
-<part name="SLOT14" library="24x16_RGB_Bottom" deviceset="SLOT" device="">
+<part name="SLOT14" library="24x16_RGB_Top" deviceset="SLOT" device="">
 <attribute name="MF" value=""/>
 <attribute name="MPN" value=""/>
 <attribute name="OC_NEWARK" value="unknown"/>
 </part>
-<part name="SLOT15" library="24x16_RGB_Bottom" deviceset="SLOT" device="">
+<part name="SLOT15" library="24x16_RGB_Top" deviceset="SLOT" device="">
 <attribute name="MF" value=""/>
 <attribute name="MPN" value=""/>
 <attribute name="OC_NEWARK" value="unknown"/>
 </part>
-<part name="SLOT16" library="24x16_RGB_Bottom" deviceset="SLOT" device="">
+<part name="SLOT16" library="24x16_RGB_Top" deviceset="SLOT" device="">
 <attribute name="MF" value=""/>
 <attribute name="MPN" value=""/>

Commit message: 
Connections:
- net MODE: no longer JP2.4
- net RST: no longer JP2.3
- net VCC: now also JP2.3, JP2.4
Changed lines of the file:
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@@
 <pinref part="JP2" gate="G$1" pin="6"/>
-</segment>
-<segment>
-<wire x1="5.08" y1="76.2" x2="20.32" y2="76.2" width="0.1524" layer="91"/>
-<pinref part="JP2" gate="G$1" pin="4"/>
-<label x="12.7" y="76.2" size="1.778" layer="95"/>
 </segment>
 </net>
@@
 <label x="12.7" y="68.58" size="1.778" layer="95"/>
 <pinref part="JP2" gate="G$1" pin="1"/>
-</segment>
-<segment>
-<wire x1="5.08" y1="73.66" x2="20.32" y2="73.66" width="0.1524" layer="91"/>
-<pinref part="JP2" gate="G$1" pin="3"/>
-<label x="12.7" y="73.66" size="1.778" layer="95"/>
 </segment>
 </net>
@@
 </segment>
 </net>
+<net name="VCC" class="0">
+<segment>
+<pinref part="JP2" gate="G$1" pin="4"/>
+<wire x1="5.08" y1="76.2" x2="20.32" y2="76.2" width="0.1524" layer="91"/>
+<label x="12.7" y="76.2" size="1.778" layer="95"/>
+</segment>
+<segment>
+<pinref part="JP2" gate="G$1" pin="3"/>
+<wire x1="5.08" y1="73.66" x2="20.32" y2="73.66" width="0.1524" layer="91"/>
+<label x="12.7" y="73.66" size="1.778" layer="95"/>
+</segment>
+</net>
