File: NSLU_USB_Boost/USB_Boost.sch (EAGLE design)
At the start: 12 parts, among them IC2 IC_TPS6120XQFN10, X1 USBKUSBX-SMT-AS1N

Commit message: 
Parts:
- renumbered BAT2 to BAT1, C62 to C1, C63 to C2, C64 to C3, IC2 to IC1, JP3 to JP1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
