File: LayerOne_2014/badge/stm32-prox/rev3/sam7/STM32-PROX.sch (EAGLE design)
At the start: 268 parts, among them IC1 IC_TPS6120XQFN10, IC10 74XX244, IC105 MCP1824T-250, IC106 MCP1824T-120, IC11 CD4066, IC12 AT91SAM7S512B, IC13 PQ1X331M2ZP-3V3-LDO-SOT-23-5, IC14 AD8052, IC3 PQ1X331M2ZP-3V3-LDO-SOT-23-5, IC4 HCU-INVERTER, IC5 TLV3502, IC6 MCP6294, IC7 MCP100, IC8 TLC5540, IC9 74XX244, K1 5-XX, K2 5-XX, K3 5-XX, Q1 NPN-SOT23-2N3904, Q3 MMBT2222, U1 FERRITE0805, U2 XC3S50, U3 UG-2864HSWEG01, U4 SDCARD, U40 BITFURY, Y1 16Mhz

Commit message: 
Parts:
- TP28, TP36, TP7: PARTNO (none) -> NONE
Changed lines of the file:
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@@
 <part name="TP25" library="STM32-PROX" deviceset="TESTPAD" device=""/>
 <part name="TP26" library="STM32-PROX" deviceset="TESTPAD" device=""/>
-<part name="TP28" library="STM32-PROX" deviceset="TESTPAD" device=""/>
+<part name="TP28" library="STM32-PROX" deviceset="TESTPAD" device="">
+<attribute name="PARTNO" value="NONE"/>
+</part>
 <part name="TP29" library="STM32-PROX" deviceset="TESTPAD" device=""/>
 <part name="TP30" library="STM32-PROX" deviceset="TESTPAD" device=""/>
@@
 <part name="TP34" library="STM32-PROX" deviceset="TESTPAD" device=""/>
 <part name="TP35" library="STM32-PROX" deviceset="TESTPAD" device=""/>
-<part name="TP36" library="STM32-PROX" deviceset="TESTPAD" device=""/>
+<part name="TP36" library="STM32-PROX" deviceset="TESTPAD" device="">
+<attribute name="PARTNO" value="NONE"/>
+</part>
 <part name="TP37" library="STM32-PROX" deviceset="TESTPAD" device=""/>
 <part name="TP38" library="STM32-PROX" deviceset="TESTPAD" device=""/>
@@
 <attribute name="PARTNO" value="GRM188R71H102KA01D"/>
 </part>
-<part name="TP7" library="STM32-PROX" deviceset="TESTPAD" device=""/>
+<part name="TP7" library="STM32-PROX" deviceset="TESTPAD" device="">
+<attribute name="PARTNO" value="NONE"/>
+</part>
 <part name="TP11" library="STM32-PROX" deviceset="TESTPAD" device=""/>
 <part name="R4" library="STM32-PROX" deviceset="RESISTOR" device="0603" value="10K">
@@
 <instance part="TP25" gate="G$1" x="33.02" y="-30.48" rot="R270"/>
 <instance part="TP26" gate="G$1" x="38.1" y="-33.02" rot="R270"/>
-<instance part="TP28" gate="G$1" x="33.02" y="40.64" rot="R270"/>
+<instance part="TP28" gate="G$1" x="33.02" y="40.64" rot="R270">
+<attribute name="PARTNO" x="33.02" y="40.64" size="1.778" layer="96" rot="R270" display="off"/>
+</instance>
 <instance part="TP29" gate="G$1" x="33.02" y="35.56" rot="R270"/>
 <instance part="TP30" gate="G$1" x="33.02" y="25.4" rot="R270"/>
@@
 <instance part="TP34" gate="G$1" x="33.02" y="5.08" rot="R270"/>
 <instance part="TP35" gate="G$1" x="33.02" y="-25.4" rot="R270"/>
-<instance part="TP36" gate="G$1" x="38.1" y="43.18" rot="R270"/>
+<instance part="TP36" gate="G$1" x="38.1" y="43.18" rot="R270">
+<attribute name="PARTNO" x="38.1" y="43.18" size="1.778" layer="96" rot="R270" display="off"/>
+</instance>
 <instance part="TP37" gate="G$1" x="38.1" y="12.7" rot="R270"/>
 <instance part="TP38" gate="G$1" x="33.02" y="10.16" rot="R270"/>
@@
 <attribute name="DIGIKEY" x="17.78" y="66.04" size="1.778" layer="96" rot="R180" display="off"/>
 </instance>
-<instance part="TP7" gate="G$1" x="38.1" y="38.1" rot="R270"/>
+<instance part="TP7" gate="G$1" x="38.1" y="38.1" rot="R270">
+<attribute name="PARTNO" x="38.1" y="38.1" size="1.778" layer="96" rot="R270" display="off"/>
+</instance>
 <instance part="TP11" gate="G$1" x="33.02" y="30.48" rot="R270"/>
 <instance part="R4" gate="G$1" x="-55.88" y="88.9" rot="R270">

Commit message: L2 CDRH2D18/HPNP-2R2NC
Parts:
- L2: DIGIKEY (none) -> 308-2295-1-ND; MF (none) -> CDRH2D18/HPNP-2R2NC; MPN (none) -> CDRH2D18/HPNP-2R2NC; PARTNO * -> CDRH2D18/HPNP-2R2NC
Changed lines of the file:
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@@
 </part>
 <part name="L2" library="STM32-PROX" deviceset="CDRH2D18" device="" value="CDRH2D18/HPNP-2R2NC">
-<attribute name="MF" value=""/>
-<attribute name="MPN" value=""/>
-<attribute name="OC_NEWARK" value="unknown"/>
-<attribute name="PARTNO" value="*"/>
+<attribute name="DIGIKEY" value="308-2295-1-ND"/>
+<attribute name="MF" value="CDRH2D18/HPNP-2R2NC"/>
+<attribute name="MPN" value="CDRH2D18/HPNP-2R2NC"/>
+<attribute name="OC_NEWARK" value="unknown"/>
+<attribute name="PARTNO" value="CDRH2D18/HPNP-2R2NC"/>
 </part>
 <part name="U$9" library="STM32-PROX" deviceset="BATT" device="">
@@
 <attribute name="MF" x="-2.54" y="22.86" size="1.778" layer="96" display="off"/>
 <attribute name="MPN" x="-2.54" y="22.86" size="1.778" layer="96" display="off"/>
+<attribute name="DIGIKEY" x="-2.54" y="22.86" size="1.778" layer="96" display="off"/>
 </instance>
 <instance part="U$9" gate="G$1" x="99.06" y="66.04">

Commit message: BZX84C47-7-F D10
Parts:
- D10: DIGIKEY (none) -> BZX84C47-FDICT-ND; MF (none) -> BZX84C47-7-F; MPN (none) -> BZX84C47-7-F; PARTNO * -> BZX84C47-7-F
- D11: DIGIKEY (none) -> BZX84C47-FDICT-ND
- D7: MF (none) -> BZX84C47-7-F; MPN (none) -> BZX84C47-7-F; PARTNO * -> BZX84C47-7-F
Changed lines of the file:
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@@
 <part name="D7" library="STM32-PROX" deviceset="DIODE-SMD-SOT23" device="">
 <attribute name="DIGIKEY" value="BZX84C47-FDICT-ND"/>
-<attribute name="MF" value=""/>
-<attribute name="MPN" value=""/>
+<attribute name="MF" value="BZX84C47-7-F"/>
+<attribute name="MPN" value="BZX84C47-7-F"/>
 <attribute name="OC_NEWARK" value="unknown"/>
-<attribute name="PARTNO" value="*"/>
+<attribute name="PARTNO" value="BZX84C47-7-F"/>
 </part>
 <part name="VDD9" library="STM32-PROX" deviceset="VDD" device=""/>
@@
 </part>
 <part name="D10" library="STM32-PROX" deviceset="DIODE-SMD-SOT23" device="">
-<attribute name="MF" value=""/>
-<attribute name="MPN" value=""/>
+<attribute name="DIGIKEY" value="BZX84C47-FDICT-ND"/>
+<attribute name="MF" value="BZX84C47-7-F"/>
+<attribute name="MPN" value="BZX84C47-7-F"/>
 <attribute name="OC_NEWARK" value="unknown"/>
-<attribute name="PARTNO" value="*"/>
+<attribute name="PARTNO" value="BZX84C47-7-F"/>
 </part>
 <part name="D11" library="STM32-PROX" deviceset="DIODE-SMD-SOT23" device="">
+<attribute name="DIGIKEY" value="BZX84C47-FDICT-ND"/>
 <attribute name="MF" value=""/>
 <attribute name="MPN" value=""/>
@@
 <attribute name="MF" x="66.04" y="-12.7" size="1.778" layer="96" display="off"/>
 <attribute name="MPN" x="66.04" y="-12.7" size="1.778" layer="96" display="off"/>
+<attribute name="DIGIKEY" x="66.04" y="-12.7" size="1.778" layer="96" rot="R90" display="off"/>
 </instance>
 <instance part="D11" gate="G$1" x="81.28" y="73.66" rot="R90">
@@
 <attribute name="MF" x="81.28" y="73.66" size="1.778" layer="96" display="off"/>
 <attribute name="MPN" x="81.28" y="73.66" size="1.778" layer="96" display="off"/>
+<attribute name="DIGIKEY" x="81.28" y="73.66" size="1.778" layer="96" rot="R90" display="off"/>
 </instance>
 <instance part="V56" gate="G$1" x="81.28" y="63.5"/>

Commit message: fb'S 600 OHM
Parts:
- FB1, FB2, FB3: value FERRITERLC_0603 -> 600 OHM
Changed lines of the file:
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@@
 <attribute name="PARTNO" value="CL10B104KO8NNNC"/>
 </part>
-<part name="FB2" library="STM32-PROX" deviceset="FERRITE" device="RLC_0603">
+<part name="FB2" library="STM32-PROX" deviceset="FERRITE" device="RLC_0603" value="600 OHM ">
 <attribute name="DIGIKEY" value="1276-6379-2-ND"/>
 <attribute name="PARTNO" value="CIM10J601NC"/>
 </part>
-<part name="FB3" library="STM32-PROX" deviceset="FERRITE" device="RLC_0603">
+<part name="FB3" library="STM32-PROX" deviceset="FERRITE" device="RLC_0603" value="600 OHM ">
 <attribute name="DIGIKEY" value="1276-6379-2-ND"/>
 <attribute name="PARTNO" value="CIM10J601NC"/>
 </part>
-<part name="FB1" library="STM32-PROX" deviceset="FERRITE" device="RLC_0603">
+<part name="FB1" library="STM32-PROX" deviceset="FERRITE" device="RLC_0603" value="600 OHM ">
 <attribute name="DIGIKEY" value="1276-6379-2-ND"/>
 <attribute name="PARTNO" value="CIM10J601NC"/>

Commit message: TESTPADS SET TO NONE
Parts:
- D11: MF (none) -> BZX84C47-7-F; MPN (none) -> BZX84C47-7-F; PARTNO * -> BZX84C47-7-F
- IC4: MPN (none) -> NC7SZ04M5X; PARTNO * -> NC7SZ04M5X
- OE1, OE10, OE11, OE2, OE3, OE4, OE5, OE6, OE7, OE8, OE9, TP1, TP2, TP3, TP4, TP5, TP_ADC_NOE: PARTNO * -> NONE
- TP11, TP12, TP13, TP14, TP15, TP16, TP18, TP19, TP20, TP22, TP23, TP24, TP25, TP26, TP29, TP30, TP31, TP32, TP33, TP34, TP35, TP37, TP38, TP39, TP40, TP42, TP43, TP44, TP45, TP46, TP47, TP48, TP49, TP50, TP51, TP52, TP53, TP54, TP55, TP56, TP6: PARTNO (none) -> NONE

Commit message: HIROSE PARTS MQ172X-4PA(66)
Parts:
- SV2: MPN (none) -> MQ172X-4PA(66); PARTNO * -> MQ172X-4PA(66)
Changed lines of the file:
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@@
 <attribute name="DIGIKEY" value="H10488CT-ND"/>
 <attribute name="MF" value="MQ172X-4PA(66)"/>
-<attribute name="MPN" value=""/>
+<attribute name="MPN" value="MQ172X-4PA(66)"/>
 <attribute name="OC_NEWARK" value="unknown"/>
-<attribute name="PARTNO" value="*"/>
+<attribute name="PARTNO" value="MQ172X-4PA(66)"/>
 </part>
 <part name="IC9" library="STM32-PROX" deviceset="74XX244-OCTAL-TRISTATE-BUFFERS" device="" value="74XX244">

Commit message: usb protection diode added D6 PRTR5V0U2X,215
Parts:
- D6: DIGIKEY (none) -> 568-4140-1-ND; MPN (none) -> PRTR5V0U2X,215; PARTNO (none) -> PRTR5V0U2X,215
Changed lines of the file:
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@@
 </part>
 <part name="V3" library="STM32-PROX" deviceset="GND" device=""/>
-<part name="D6" library="badge.lbrbadge_2013" deviceset="USBUG_PRTR5V0U2X" device=""/>
+<part name="D6" library="badge.lbrbadge_2013" deviceset="USBUG_PRTR5V0U2X" device="">
+<attribute name="DIGIKEY" value="568-4140-1-ND"/>
+<attribute name="MPN" value="PRTR5V0U2X,215"/>
+<attribute name="PARTNO" value="PRTR5V0U2X,215"/>
+</part>
 <part name="V5" library="STM32-PROX" deviceset="GND" device=""/>
 <part name="TP16" library="STM32-PROX" deviceset="TESTPAD" device="">
@@
 </instance>
 <instance part="V3" gate="G$1" x="-27.94" y="76.2" rot="R90"/>
-<instance part="D6" gate="G$1" x="-15.24" y="38.1"/>
+<instance part="D6" gate="G$1" x="-15.24" y="38.1">
+<attribute name="MPN" x="-15.24" y="38.1" size="1.778" layer="96" display="off"/>
+<attribute name="PARTNO" x="-15.24" y="38.1" size="1.778" layer="96" display="off"/>
+<attribute name="DIGIKEY" x="-15.24" y="38.1" size="1.778" layer="96" display="off"/>
+</instance>
 <instance part="V5" gate="G$1" x="-20.32" y="22.86"/>
 <instance part="TP18" gate="G$1" x="134.62" y="33.02">

Commit message: buz1 part CCV-084B16-SMT added
Parts:
- BUZ1: DIGIKEY (none) -> 102-1265-2-ND; MF (none) -> CUI Inc; MPN (none) -> CCV-084B16-SMT; PARTNO (none) -> CCV-084B16-SMT
Changed lines of the file:
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@@
 <attribute name="PARTNO" value="NONE"/>
 </part>
-<part name="BUZ1" library="STM32-PROX" deviceset="BUZZER" device=""/>
+<part name="BUZ1" library="STM32-PROX" deviceset="BUZZER" device="">
+<attribute name="DIGIKEY" value="102-1265-2-ND"/>
+<attribute name="MF" value="CUI Inc"/>
+<attribute name="MPN" value="CCV-084B16-SMT"/>
+<attribute name="PARTNO" value="CCV-084B16-SMT"/>
+</part>
 </parts>
 <sheets>
@@
 <attribute name="DIGIKEY" x="-55.88" y="88.9" size="1.778" layer="96" rot="R270" display="off"/>
 </instance>
-<instance part="BUZ1" gate="G$1" x="-115.57" y="-7.62"/>
+<instance part="BUZ1" gate="G$1" x="-115.57" y="-7.62">
+<attribute name="MF" x="-115.57" y="-7.62" size="1.778" layer="96" display="off"/>
+<attribute name="MPN" x="-115.57" y="-7.62" size="1.778" layer="96" display="off"/>
+<attribute name="PARTNO" x="-115.57" y="-7.62" size="1.778" layer="96" display="off"/>
+<attribute name="DIGIKEY" x="-115.57" y="-7.62" size="1.778" layer="96" display="off"/>
+</instance>
 </instances>
 <busses>
