File: ZTable/trunk/eagle/zTable.sch (EAGLE design)
At the start: 16 parts

Commit message: 
Parts:
- R0, R1, R2, R3, R4, R5, R6, R7, R8: device SparkFun:RESISTOR0603-RES -> SparkFun:RESISTOR
Changed lines of the file:
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@@
 <part name="C1" library="SparkFun" deviceset="CAP" device="0805" value="0.1uF"/>
 <part name="SUPPLY2" library="supply2" deviceset="GND" device=""/>
-<part name="R0" library="SparkFun" deviceset="RESISTOR" device="0603-RES" value="16"/>
+<part name="R0" library="SparkFun" deviceset="RESISTOR" device="" value="16"/>
 <part name="OPT1" library="SparkFun" deviceset="JUMPER-2" device="PTH"/>
-<part name="R1" library="SparkFun" deviceset="RESISTOR" device="0603-RES" value="16"/>
-<part name="R2" library="SparkFun" deviceset="RESISTOR" device="0603-RES" value="16"/>
-<part name="R3" library="SparkFun" deviceset="RESISTOR" device="0603-RES" value="16"/>
-<part name="R4" library="SparkFun" deviceset="RESISTOR" device="0603-RES" value="16"/>
-<part name="R5" library="SparkFun" deviceset="RESISTOR" device="0603-RES" value="16"/>
-<part name="R6" library="SparkFun" deviceset="RESISTOR" device="0603-RES" value="16"/>
-<part name="R7" library="SparkFun" deviceset="RESISTOR" device="0603-RES" value="16"/>
-<part name="R8" library="SparkFun" deviceset="RESISTOR" device="0603-RES" value="16"/>
+<part name="R1" library="SparkFun" deviceset="RESISTOR" device="" value="16"/>
+<part name="R2" library="SparkFun" deviceset="RESISTOR" device="" value="16"/>
+<part name="R3" library="SparkFun" deviceset="RESISTOR" device="" value="16"/>
+<part name="R4" library="SparkFun" deviceset="RESISTOR" device="" value="16"/>
+<part name="R5" library="SparkFun" deviceset="RESISTOR" device="" value="16"/>
+<part name="R6" library="SparkFun" deviceset="RESISTOR" device="" value="16"/>
+<part name="R7" library="SparkFun" deviceset="RESISTOR" device="" value="16"/>
+<part name="R8" library="SparkFun" deviceset="RESISTOR" device="" value="16"/>
 <part name="OPT2" library="SparkFun" deviceset="JUMPER-2" device="PTH"/>
 <part name="SUPPLY5" library="supply2" deviceset="GND" device=""/>
