File: LayerOne_2015/Demoscene/PCB/L1Demoscene_v2.sch (EAGLE design)
At the start: 58 parts, among them IC1 MEGA8-AI, IC2 REG1117, J1 AVR_SPI_PRG_6PTH, J2 CON_HEADER_1X02-PTH, J3 CON_HEADER_2X04-PTH

Commit message: 
Parts:
- removed JP3: USB-MICROB, STM32-PROX:USB-MICROB
- added U1: (no value), SparkFun-Connectors:USB-ABCONN-11794
- 10K: value (none) -> R34
- R30, R31, R32, R33: value 1k -> 10k
- S1: value Switch -> Reset
- S2: value Switch -> User Switch
Connections:
- net GND: now also U1.GND; no longer JP3.GND
- net VIN: now also U1.VBUS; no longer JP3.VBUS
Changed lines of the file:
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@@
 <layer number="54" name="bGND_GNDA" color="1" fill="9" visible="no" active="no"/>
 <layer number="56" name="wert" color="7" fill="1" visible="no" active="no"/>
+<layer number="57" name="tCAD" color="7" fill="1" visible="no" active="no"/>
 <layer number="91" name="Nets" color="2" fill="1" visible="yes" active="yes"/>
 <layer number="92" name="Busses" color="1" fill="1" visible="yes" active="yes"/>
@@
 <layer number="97" name="Info" color="7" fill="1" visible="yes" active="yes"/>
 <layer number="98" name="Guide" color="6" fill="1" visible="yes" active="yes"/>
+<layer number="99" name="SpiceOrder" color="7" fill="1" visible="yes" active="yes"/>
 <layer number="100" name="Muster" color="7" fill="1" visible="no" active="no"/>
 <layer number="101" name="Patch_Top" color="12" fill="4" visible="no" active="yes"/>
@@
 <layer number="151" name="HeatSink" color="7" fill="1" visible="no" active="yes"/>
 <layer number="152" name="_bDocu" color="7" fill="1" visible="no" active="yes"/>
+<layer number="153" name="FabDoc1" color="7" fill="1" visible="no" active="yes"/>
+<layer number="154" name="FabDoc2" color="7" fill="1" visible="no" active="yes"/>
+<layer number="155" name="FabDoc3" color="7" fill="1" visible="no" active="yes"/>
 <layer number="191" name="mNets" color="7" fill="1" visible="no" active="yes"/>
 <layer number="192" name="mBusses" color="7" fill="1" visible="no" active="yes"/>
@@
 <part name="C3" library="SparkFun-Capacitors" deviceset="CAP_POL" device="1206"/>
 <part name="J1" library="SparkFun-Connectors" deviceset="AVR_SPI_PRG_6" device="PTH"/>
-<part name="10K" library="SparkFun-Resistors" deviceset="RESISTOR" device="0603-RES"/>
+<part name="10K" library="SparkFun-Resistors" deviceset="RESISTOR" device="0603-RES" value="R34"/>
 <part name="SUPPLY3" library="SparkFun-Aesthetics" deviceset="VCC" device=""/>
 <part name="SUPPLY4" library="SparkFun-Aesthetics" deviceset="VCC" device=""/>
@@
 <part name="JP1" library="SparkFun-Connectors" deviceset="AUDIO-JACK" device="PTH"/>
 <part name="GND11" library="SparkFun-Aesthetics" deviceset="GND" device=""/>
-<part name="JP3" library="STM32-PROX" deviceset="USB" device="-MICROB"/>
 <part name="GND12" library="SparkFun-Aesthetics" deviceset="GND" device=""/>
 <part name="R27" library="SparkFun-Resistors" deviceset="RESISTOR" device="0603-RES" value="1k"/>
@@
 <part name="C4" library="dp_devices" deviceset="CAPACITOR_POL" device="-SMC_A"/>
 <part name="C5" library="dp_devices" deviceset="CAPACITOR_POL" device="-SMC_A"/>
-<part name="S1" library="tvbgone-2layer" deviceset="SPARKFUN-ELECTROMECHANICAL_SWITCH-MOMENTARY-2" device="-SMD-1101NE" value="Switch"/>
+<part name="S1" library="tvbgone-2layer" deviceset="SPARKFUN-ELECTROMECHANICAL_SWITCH-MOMENTARY-2" device="-SMD-1101NE" value="Reset"/>
 <part name="GND15" library="SparkFun-Aesthetics" deviceset="GND" device=""/>
 <part name="C6" library="SparkFun-Capacitors" deviceset="CAP" device="0603-CAP" value="100nf"/>
@@
 <part name="LED1" library="dp_devices" deviceset="LED" device="-0603"/>
 <part name="GND18" library="SparkFun-Aesthetics" deviceset="GND" device=""/>
-<part name="S2" library="tvbgone-2layer" deviceset="SPARKFUN-ELECTROMECHANICAL_SWITCH-MOMENTARY-2" device="-SMD-1101NE" value="Switch"/>
+<part name="S2" library="tvbgone-2layer" deviceset="SPARKFUN-ELECTROMECHANICAL_SWITCH-MOMENTARY-2" device="-SMD-1101NE" value="User Switch"/>
 <part name="GND19" library="SparkFun-Aesthetics" deviceset="GND" device=""/>
 <part name="J3" library="dp_devices" deviceset="CON_HEADER_2X04" device="-PTH"/>
-<part name="R30" library="SparkFun-Resistors" deviceset="RESISTOR" device="0603-RES" value="1k"/>
-<part name="R31" library="SparkFun-Resistors" deviceset="RESISTOR" device="0603-RES" value="1k"/>
-<part name="R32" library="SparkFun-Resistors" deviceset="RESISTOR" device="0603-RES" value="1k"/>
-<part name="R33" library="SparkFun-Resistors" deviceset="RESISTOR" device="0603-RES" value="1k"/>
+<part name="R30" library="SparkFun-Resistors" deviceset="RESISTOR" device="0603-RES" value="10k"/>
+<part name="R31" library="SparkFun-Resistors" deviceset="RESISTOR" device="0603-RES" value="10k"/>
+<part name="R32" library="SparkFun-Resistors" deviceset="RESISTOR" device="0603-RES" value="10k"/>
+<part name="R33" library="SparkFun-Resistors" deviceset="RESISTOR" device="0603-RES" value="10k"/>
 <part name="GND20" library="SparkFun-Aesthetics" deviceset="GND" device=""/>
 <part name="SUPPLY7" library="SparkFun-Aesthetics" deviceset="VCC" device=""/>
+<part name="U1" library="SparkFun-Connectors" deviceset="USB-AB" device="CONN-11794"/>
 </parts>
 <sheets>
@@
 <instance part="JP1" gate="G$1" x="317.5" y="38.1" rot="R180"/>
 <instance part="GND11" gate="1" x="307.34" y="30.48"/>
-<instance part="JP3" gate="G$1" x="190.5" y="-20.32"/>
-<instance part="GND12" gate="1" x="185.42" y="-25.4"/>
+<instance part="GND12" gate="1" x="195.58" y="-2.54" rot="R180"/>
 <instance part="R27" gate="G$1" x="142.24" y="22.86" rot="R90"/>
 <instance part="PWR" gate="LED" x="142.24" y="12.7"/>
@@
 <instance part="GND20" gate="1" x="391.16" y="160.02"/>
 <instance part="SUPPLY7" gate="1" x="360.68" y="147.32" rot="R180"/>
+<instance part="U1" gate="G$1" x="205.74" y="-15.24"/>
 </instances>
 <busses>
@@
 <wire x1="347.98" y1="101.6" x2="360.68" y2="101.6" width="0.1524" layer="91"/>
 <label x="355.6" y="101.6" size="1.778" layer="95"/>
-</segment>
-<segment>
-<pinref part="JP3" gate="G$1" pin="GND"/>
-<pinref part="GND12" gate="1" pin="GND"/>
-<wire x1="187.96" y1="-20.32" x2="185.42" y2="-20.32" width="0.1524" layer="91"/>
-<wire x1="185.42" y1="-20.32" x2="185.42" y2="-22.86" width="0.1524" layer="91"/>
 </segment>
 <segment>
@@
 <pinref part="J3" gate="G$1" pin="P$8"/>
 <wire x1="386.08" y1="170.18" x2="391.16" y2="170.18" width="0.1524" layer="91"/>
+</segment>
+<segment>
+<pinref part="GND12" gate="1" pin="GND"/>
+<pinref part="U1" gate="G$1" pin="GND"/>
+<wire x1="195.58" y1="-5.08" x2="195.58" y2="-10.16" width="0.1524" layer="91"/>
+<wire x1="195.58" y1="-10.16" x2="200.66" y2="-10.16" width="0.1524" layer="91"/>
 </segment>
 </net>
@@
 <net name="VIN" class="0">
 <segment>
-<pinref part="JP3" gate="G$1" pin="VBUS"/>
 <pinref part="IC2" gate="G$1" pin="VIN"/>
 <wire x1="187.96" y1="-17.78" x2="180.34" y2="-17.78" width="0.1524" layer="91"/>
@@
 <junction x="180.34" y="-17.78"/>
 <label x="180.34" y="-15.24" size="1.778" layer="95"/>
-</segment>
-<segment>
+<pinref part="U1" gate="G$1" pin="VBUS"/>
+<wire x1="187.96" y1="-17.78" x2="187.96" y2="-20.32" width="0.1524" layer="91"/>
+<wire x1="187.96" y1="-20.32" x2="200.66" y2="-20.32" width="0.1524" layer="91"/>
+</segment>
+<segment>

Commit message: 
Parts:
- removed U1: (no value), SparkFun-Connectors:USB-ABCONN-11794
- added X1: USB-MICROB, STM32-PROX:USB-MICROB
Connections:
- net GND: now also X1.GND; no longer U1.GND
- net VIN: now also X1.VBUS; no longer U1.VBUS
Changed lines of the file:
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@@
 <part name="GND20" library="SparkFun-Aesthetics" deviceset="GND" device=""/>
 <part name="SUPPLY7" library="SparkFun-Aesthetics" deviceset="VCC" device=""/>
-<part name="U1" library="SparkFun-Connectors" deviceset="USB-AB" device="CONN-11794"/>
+<part name="X1" library="STM32-PROX" deviceset="USB" device="-MICROB"/>
 </parts>
 <sheets>
@@
 <instance part="GND20" gate="1" x="391.16" y="160.02"/>
 <instance part="SUPPLY7" gate="1" x="360.68" y="147.32" rot="R180"/>
-<instance part="U1" gate="G$1" x="205.74" y="-15.24"/>
+<instance part="X1" gate="G$1" x="203.2" y="-10.16" rot="MR180"/>
 </instances>
 <busses>
@@
 <segment>
 <pinref part="GND12" gate="1" pin="GND"/>
-<pinref part="U1" gate="G$1" pin="GND"/>
 <wire x1="195.58" y1="-5.08" x2="195.58" y2="-10.16" width="0.1524" layer="91"/>
 <wire x1="195.58" y1="-10.16" x2="200.66" y2="-10.16" width="0.1524" layer="91"/>
+<pinref part="X1" gate="G$1" pin="GND"/>
 </segment>
 </net>
@@
 <junction x="180.34" y="-17.78"/>
 <label x="180.34" y="-15.24" size="1.778" layer="95"/>
-<pinref part="U1" gate="G$1" pin="VBUS"/>
-<wire x1="187.96" y1="-17.78" x2="187.96" y2="-20.32" width="0.1524" layer="91"/>
-<wire x1="187.96" y1="-20.32" x2="200.66" y2="-20.32" width="0.1524" layer="91"/>
-</segment>
-<segment>
+<wire x1="187.96" y1="-17.78" x2="195.58" y2="-17.78" width="0.1524" layer="91"/>
+<wire x1="195.58" y1="-17.78" x2="195.58" y2="-12.7" width="0.1524" layer="91"/>
+<pinref part="X1" gate="G$1" pin="VBUS"/>
+<wire x1="195.58" y1="-12.7" x2="200.66" y2="-12.7" width="0.1524" layer="91"/>
+</segment>
+<segment>
