File: LayerOne_2015/Demoscene/PCB/L1Demoscene_v3.sch (EAGLE design)
At the start: 40 parts, among them IC2 REG1117, J1 CON_HEADER_1X02-PTH, J2 CON_HEADER_1X02-PTH, J3 CON_HEADER_2X04-PTH, U2 PIC24FXXXDAX06

Commit message: Added Crystal and removed USBID switch
Parts:
- removed LED1: (no value), SparkFun-LED:LED0603
- removed R4: 750, SparkFun-Resistors:RESISTOR0603-RES
- removed S1: (no value), SparkFun-Electromechanical:SWITCH-SPDT-SMD-A
- added C6, C7: 9pF, SparkFun-Capacitors:CAP0603-CAP
- added Y1: (no value), SparkFun-FreqCtrl:CRYSTAL5X3
Connections:
- removed net BOOT: LED1.C, U2.OSCI/CLKI/CN23/RC12
- new net N$20: C6.1, U2.OSCO/CLKO/CN22/RC15, Y1.2
- net 3.3V: no longer R4.2
- net GND: now also C6.2, C7.2; no longer S1.O
- net N$3: now also C7.1, U2.OSCI/CLKI/CN23/RC12, Y1.1; no longer LED1.A, R4.1
- net USBID: no longer S1.P
Changed lines of the file:
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@@
 <part name="SUPPLY2" library="SparkFun-Aesthetics" deviceset="3.3V" device=""/>
 <part name="SUPPLY3" library="SparkFun-Aesthetics" deviceset="3.3V" device=""/>
-<part name="SUPPLY4" library="SparkFun-Aesthetics" deviceset="3.3V" device=""/>
 <part name="SUPPLY8" library="SparkFun-Aesthetics" deviceset="3.3V" device=""/>
 <part name="GND1" library="SparkFun-Aesthetics" deviceset="GND" device=""/>
@@
 <part name="R2" library="SparkFun-Resistors" deviceset="RESISTOR" device="0603-RES" value="10K"/>
 <part name="R3" library="SparkFun-Resistors" deviceset="RESISTOR" device="0603-RES" value="470"/>
-<part name="R4" library="SparkFun-Resistors" deviceset="RESISTOR" device="0603-RES" value="750"/>
 <part name="GND5" library="SparkFun-Aesthetics" deviceset="GND" device=""/>
 <part name="GND6" library="SparkFun-Aesthetics" deviceset="GND" device=""/>
-<part name="S1" library="SparkFun-Electromechanical" deviceset="SWITCH-SPDT" device="-SMD-A"/>
-<part name="GND7" library="SparkFun-Aesthetics" deviceset="GND" device=""/>
-<part name="LED1" library="SparkFun-LED" deviceset="LED" device="0603"/>
 <part name="C2" library="SparkFun-Capacitors" deviceset="CAP_POL" device="1206" value="10uF"/>
 <part name="GND8" library="SparkFun-Aesthetics" deviceset="GND" device=""/>
@@
 <part name="R1" library="SparkFun-Resistors" deviceset="RESISTOR" device="0603-RES" value="2K"/>
 <part name="GND16" library="SparkFun-Aesthetics" deviceset="GND" device=""/>
+<part name="Y1" library="SparkFun-FreqCtrl" deviceset="CRYSTAL" device="5X3"/>
+<part name="C6" library="SparkFun-Capacitors" deviceset="CAP" device="0603-CAP" value="9pF"/>
+<part name="C7" library="SparkFun-Capacitors" deviceset="CAP" device="0603-CAP" value="9pF"/>
+<part name="GND18" library="SparkFun-Aesthetics" deviceset="GND" device=""/>
+<part name="GND19" library="SparkFun-Aesthetics" deviceset="GND" device=""/>
 </parts>
 <sheets>
@@
 <instance part="SUPPLY2" gate="G$1" x="73.66" y="254"/>
 <instance part="SUPPLY3" gate="G$1" x="78.74" y="289.56"/>
-<instance part="SUPPLY4" gate="G$1" x="175.26" y="215.9"/>
 <instance part="SUPPLY8" gate="G$1" x="162.56" y="170.18"/>
 <instance part="GND1" gate="1" x="45.72" y="119.38"/>
@@
 <instance part="R2" gate="G$1" x="78.74" y="281.94" rot="R90"/>
 <instance part="R3" gate="G$1" x="78.74" y="266.7" rot="R90"/>
-<instance part="R4" gate="G$1" x="175.26" y="205.74" rot="R90"/>
 <instance part="GND5" gate="1" x="162.56" y="139.7"/>
 <instance part="GND6" gate="1" x="193.04" y="149.86"/>
-<instance part="S1" gate="1" x="182.88" y="154.94" rot="R180"/>
-<instance part="GND7" gate="1" x="175.26" y="139.7"/>
-<instance part="LED1" gate="G$1" x="175.26" y="195.58"/>
 <instance part="C2" gate="G$1" x="91.44" y="256.54" rot="R90"/>
 <instance part="GND8" gate="1" x="101.6" y="256.54" rot="R90"/>
@@
 <instance part="R1" gate="G$1" x="193.04" y="287.02"/>
 <instance part="GND16" gate="1" x="182.88" y="279.4"/>
+<instance part="Y1" gate="G$1" x="203.2" y="195.58" rot="R90"/>
+<instance part="C6" gate="G$1" x="215.9" y="203.2" rot="R90"/>
+<instance part="C7" gate="G$1" x="215.9" y="187.96" rot="R90"/>
+<instance part="GND18" gate="1" x="228.6" y="203.2" rot="R90"/>
+<instance part="GND19" gate="1" x="228.6" y="187.96" rot="R90"/>
 </instances>
 <busses>
@@
 </segment>
 <segment>
-<pinref part="S1" gate="1" pin="O"/>
-<pinref part="GND7" gate="1" pin="GND"/>
-<wire x1="177.8" y1="152.4" x2="175.26" y2="152.4" width="0.1524" layer="91"/>
-<wire x1="175.26" y1="152.4" x2="175.26" y2="142.24" width="0.1524" layer="91"/>
-</segment>
-<segment>
 <pinref part="C2" gate="G$1" pin="-"/>
 <pinref part="GND8" gate="1" pin="GND"/>
@@
 <wire x1="187.96" y1="287.02" x2="182.88" y2="287.02" width="0.1524" layer="91"/>
 <wire x1="182.88" y1="287.02" x2="182.88" y2="281.94" width="0.1524" layer="91"/>
+</segment>
+<segment>
+<pinref part="C6" gate="G$1" pin="2"/>
+<pinref part="GND18" gate="1" pin="GND"/>
+<wire x1="218.44" y1="203.2" x2="226.06" y2="203.2" width="0.1524" layer="91"/>
+</segment>
+<segment>
+<pinref part="C7" gate="G$1" pin="2"/>
+<pinref part="GND19" gate="1" pin="GND"/>
+<wire x1="218.44" y1="187.96" x2="226.06" y2="187.96" width="0.1524" layer="91"/>
 </segment>
 </net>
@@
 </segment>
 <segment>
-<pinref part="R4" gate="G$1" pin="2"/>
-<pinref part="SUPPLY4" gate="G$1" pin="3.3V"/>
-<wire x1="175.26" y1="210.82" x2="175.26" y2="215.9" width="0.1524" layer="91"/>
-</segment>
-<segment>
 <pinref part="SUPPLY2" gate="G$1" pin="3.3V"/>
 <pinref part="U2" gate="G$1" pin="ENVREG"/>
@@
 <wire x1="187.96" y1="160.02" x2="200.66" y2="160.02" width="0.1524" layer="91"/>
 <label x="187.96" y="160.02" size="1.778" layer="95"/>
-<pinref part="S1" gate="1" pin="P"/>
-<wire x1="185.42" y1="154.94" x2="187.96" y2="154.94" width="0.1524" layer="91"/>
-<wire x1="187.96" y1="154.94" x2="187.96" y2="160.02" width="0.1524" layer="91"/>
 </segment>
 <segment>
@@
 <wire x1="27.94" y1="175.26" x2="15.24" y2="175.26" width="0.1524" layer="91"/>
 <label x="15.24" y="175.26" size="1.778" layer="95"/>
-</segment>
-</net>
-<net name="BOOT" class="0">
-<segment>
-<pinref part="U2" gate="G$1" pin="OSCI/CLKI/CN23/RC12"/>
-<wire x1="147.32" y1="187.96" x2="175.26" y2="187.96" width="0.1524" layer="91"/>
-<pinref part="LED1" gate="G$1" pin="C"/>
-<wire x1="175.26" y1="187.96" x2="175.26" y2="190.5" width="0.1524" layer="91"/>
-<label x="152.4" y="187.96" size="1.778" layer="95"/>
-</segment>
-</net>
-<net name="N$3" class="0">
-<segment>
-<pinref part="R4" gate="G$1" pin="1"/>
-<pinref part="LED1" gate="G$1" pin="A"/>
-<wire x1="175.26" y1="200.66" x2="175.26" y2="198.12" width="0.1524" layer="91"/>
 </segment>
 </net>
@@
 </segment>
 </net>
+<net name="N$20" class="0">
+<segment>
+<pinref part="U2" gate="G$1" pin="OSCO/CLKO/CN22/RC15"/>
+<wire x1="147.32" y1="195.58" x2="187.96" y2="195.58" width="0.1524" layer="91"/>
+<wire x1="187.96" y1="195.58" x2="187.96" y2="203.2" width="0.1524" layer="91"/>
+<pinref part="Y1" gate="G$1" pin="2"/>
+<wire x1="187.96" y1="203.2" x2="203.2" y2="203.2" width="0.1524" layer="91"/>
+<pinref part="C6" gate="G$1" pin="1"/>
+<wire x1="203.2" y1="203.2" x2="203.2" y2="198.12" width="0.1524" layer="91"/>
+<wire x1="210.82" y1="203.2" x2="203.2" y2="203.2" width="0.1524" layer="91"/>
+<junction x="203.2" y="203.2"/>
+</segment>
+</net>
+<net name="N$3" class="0">
+<segment>
+<pinref part="U2" gate="G$1" pin="OSCI/CLKI/CN23/RC12"/>
+<pinref part="Y1" gate="G$1" pin="1"/>
+<wire x1="147.32" y1="187.96" x2="203.2" y2="187.96" width="0.1524" layer="91"/>
+<wire x1="203.2" y1="187.96" x2="203.2" y2="193.04" width="0.1524" layer="91"/>
+<pinref part="C7" gate="G$1" pin="1"/>
+<wire x1="210.82" y1="187.96" x2="203.2" y2="187.96" width="0.1524" layer="91"/>
+<junction x="203.2" y="187.96"/>
+</segment>
+</net>

Commit message: Small modifications
Parts:
- C6, C7: value 9pF -> 18pF
Changed lines of the file:
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@@
 <part name="GND16" library="SparkFun-Aesthetics" deviceset="GND" device=""/>
 <part name="Y1" library="SparkFun-FreqCtrl" deviceset="CRYSTAL" device="5X3"/>
-<part name="C6" library="SparkFun-Capacitors" deviceset="CAP" device="0603-CAP" value="9pF"/>
-<part name="C7" library="SparkFun-Capacitors" deviceset="CAP" device="0603-CAP" value="9pF"/>
+<part name="C6" library="SparkFun-Capacitors" deviceset="CAP" device="0603-CAP" value="18pF"/>
+<part name="C7" library="SparkFun-Capacitors" deviceset="CAP" device="0603-CAP" value="18pF"/>
 <part name="GND18" library="SparkFun-Aesthetics" deviceset="GND" device=""/>
 <part name="GND19" library="SparkFun-Aesthetics" deviceset="GND" device=""/>

Commit message: -Set Pins 6,7,8 on the VGA connector to ground for color ground return -Added ground vias for better return paths -Added two extra pads for hackery
Parts:
- added RP21, RP26: TPTP06R, testpad:TPTP06R
Connections:
- new net TP1: RP26.TP, U2.C1INC/RP26/CN9/RG7
- new net TP2: RP21.TP, U2.C1IND/RP21/CN8/RG6
- net GND: now also U$1.6, U$1.7, U$1.8
Changed lines of the file:
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@@
 <setting verticaltext="up"/>
 </settings>
-<grid distance="0.1" unitdist="inch" unit="inch" style="lines" multiple="1" display="no" altdistance="0.01" altunitdist="inch" altunit="inch"/>
+<grid distance="0.1" unitdist="inch" unit="inch" style="lines" multiple="1" display="yes" altdistance="0.01" altunitdist="inch" altunit="inch"/>
 <layers>
 <layer number="1" name="Top" color="4" fill="1" visible="no" active="no"/>
@@
 <part name="GND18" library="SparkFun-Aesthetics" deviceset="GND" device=""/>
 <part name="GND19" library="SparkFun-Aesthetics" deviceset="GND" device=""/>
+<part name="GND7" library="SparkFun-Aesthetics" deviceset="GND" device=""/>
+<part name="RP26" library="testpad" deviceset="TP" device="TP06R"/>
+<part name="RP21" library="testpad" deviceset="TP" device="TP06R"/>
 </parts>
 <sheets>
@@
 <instance part="SUPPLY2" gate="G$1" x="73.66" y="254"/>
 <instance part="SUPPLY3" gate="G$1" x="78.74" y="289.56"/>
-<instance part="SUPPLY8" gate="G$1" x="162.56" y="170.18"/>
+<instance part="SUPPLY8" gate="G$1" x="167.64" y="160.02" rot="R270"/>
 <instance part="GND1" gate="1" x="45.72" y="119.38"/>
 <instance part="GND2" gate="1" x="55.88" y="119.38"/>
@@
 <instance part="GND18" gate="1" x="228.6" y="203.2" rot="R90"/>
 <instance part="GND19" gate="1" x="228.6" y="187.96" rot="R90"/>
+<instance part="GND7" gate="1" x="248.92" y="12.7"/>
+<instance part="RP26" gate="G$1" x="177.8" y="182.88"/>
+<instance part="RP21" gate="G$1" x="185.42" y="182.88"/>
 </instances>
 <busses>
@@
 </segment>
 <segment>
-<wire x1="254" y1="40.64" x2="253.746" y2="40.64" width="0.1524" layer="91"/>
 <label x="238.76" y="40.64" size="1.778" layer="95"/>
 <pinref part="U$1" gate="G$1" pin="10"/>
-<wire x1="253.746" y1="40.64" x2="238.76" y2="40.64" width="0.1524" layer="91"/>
-<junction x="253.746" y="40.64"/>
+<wire x1="254" y1="40.64" x2="238.76" y2="40.64" width="0.1524" layer="91"/>
+<junction x="254" y="40.64"/>
 </segment>
 <segment>
@@
 <wire x1="218.44" y1="187.96" x2="226.06" y2="187.96" width="0.1524" layer="91"/>
 </segment>
+<segment>
+<pinref part="U$1" gate="G$1" pin="8"/>
+<pinref part="GND7" gate="1" pin="GND"/>
+<wire x1="254" y1="30.48" x2="248.92" y2="30.48" width="0.1524" layer="91"/>
+<wire x1="248.92" y1="30.48" x2="248.92" y2="25.4" width="0.1524" layer="91"/>
+<pinref part="U$1" gate="G$1" pin="7"/>
+<wire x1="248.92" y1="25.4" x2="248.92" y2="20.32" width="0.1524" layer="91"/>
+<wire x1="248.92" y1="20.32" x2="248.92" y2="15.24" width="0.1524" layer="91"/>
+<wire x1="254" y1="25.4" x2="248.92" y2="25.4" width="0.1524" layer="91"/>
+<pinref part="U$1" gate="G$1" pin="6"/>
+<wire x1="254" y1="20.32" x2="248.92" y2="20.32" width="0.1524" layer="91"/>
+<junction x="248.92" y="20.32"/>
+<junction x="248.92" y="25.4"/>
+</segment>
 </net>
 <net name="HSYNC" class="0">
 <segment>
-<wire x1="254" y1="33.02" x2="253.746" y2="33.02" width="0.1524" layer="91"/>
 <label x="238.76" y="33.02" size="1.778" layer="95"/>
 <pinref part="U$1" gate="G$1" pin="13"/>
-<wire x1="253.746" y1="33.02" x2="238.76" y2="33.02" width="0.1524" layer="91"/>
-<junction x="253.746" y="33.02"/>
+<wire x1="254" y1="33.02" x2="238.76" y2="33.02" width="0.1524" layer="91"/>
+<junction x="254" y="33.02"/>
 </segment>
 <segment>
@@
 <net name="VSYNC" class="0">
 <segment>
-<wire x1="254" y1="38.1" x2="253.746" y2="38.1" width="0.1524" layer="91"/>
 <label x="238.76" y="38.1" size="1.778" layer="95"/>
 <pinref part="U$1" gate="G$1" pin="14"/>
-<wire x1="253.746" y1="38.1" x2="238.76" y2="38.1" width="0.1524" layer="91"/>
-<junction x="253.746" y="38.1"/>
+<wire x1="254" y1="38.1" x2="238.76" y2="38.1" width="0.1524" layer="91"/>
+<junction x="254" y="38.1"/>
 </segment>
 <segment>
@@
 <pinref part="SUPPLY8" gate="G$1" pin="3.3V"/>
 <wire x1="147.32" y1="160.02" x2="162.56" y2="160.02" width="0.1524" layer="91"/>
-<wire x1="162.56" y1="160.02" x2="162.56" y2="170.18" width="0.1524" layer="91"/>
+<wire x1="162.56" y1="160.02" x2="167.64" y2="160.02" width="0.1524" layer="91"/>
 <pinref part="C1" gate="G$1" pin="1"/>
 <wire x1="162.56" y1="154.94" x2="162.56" y2="160.02" width="0.1524" layer="91"/>
@@
 </segment>
 </net>
+<net name="TP2" class="0">
+<segment>
+<pinref part="U2" gate="G$1" pin="C1IND/RP21/CN8/RG6"/>
+<label x="149.86" y="172.72" size="1.778" layer="95"/>
+<pinref part="RP21" gate="G$1" pin="TP"/>
+<wire x1="147.32" y1="172.72" x2="185.42" y2="172.72" width="0.1524" layer="91"/>
+<wire x1="185.42" y1="172.72" x2="185.42" y2="180.34" width="0.1524" layer="91"/>
+</segment>
+</net>
+<net name="TP1" class="0">
+<segment>
+<pinref part="U2" gate="G$1" pin="C1INC/RP26/CN9/RG7"/>
+<label x="149.86" y="175.26" size="1.778" layer="95"/>
+<pinref part="RP26" gate="G$1" pin="TP"/>
+<wire x1="147.32" y1="175.26" x2="177.8" y2="175.26" width="0.1524" layer="91"/>
+<wire x1="177.8" y1="175.26" x2="177.8" y2="180.34" width="0.1524" layer="91"/>
+</segment>
+</net>
