File: LayerOne_2015/Badge/eagle/dock/vocore_dock.brd (EAGLE design)
At the start: 25.6 x 25.6 mm, 34 parts

Commit message: 
Parts:
- PB04, PB05, PB06, PB07, PB12, PB13, PB14, PB15, PB16, PB17, PB18, PL05, PL06, PL07, PL08, PT02, PT03, PT04: device VoCore.dock.pcb:PORT_1PIN_DECAL_1PRIMARY -> vocore_dock:PORT_1PIN_DECAL_1PRIMARY
