File: LayerOne_2016/LayerOne_2016.brd (EAGLE design)
At the start: 101 x 43.8 mm, 67 parts, among them IC1 M74VHC1GT125DF2G

Commit message: 
Parts:
- removed JP1-DOUT: (no value), adafruit:1X01-CLEANBIG
- added JP14: (no value), SparkFun-Connectors:1X03_NO_SILK
Connections:
- net GND: now also JP14.3
- net N$26: now also JP14.2; no longer JP1-DOUT.1
- net VCC: now also JP14.1
Routing:
- net VCC: track 304.0 -> 308.3 mm
- net N$47: track 0.00 -> 2.54 mm
- net N$46: track 0.00 -> 2.54 mm
- net N$49: track 0.00 -> 2.54 mm
- net N$48: track 0.00 -> 2.54 mm
- net N$41: track 0.00 -> 2.54 mm
- net N$40: track 0.00 -> 2.54 mm
- net N$39: track 0.00 -> 2.54 mm
- net N$38: track 0.00 -> 2.54 mm
- net N$37: track 0.00 -> 2.54 mm
- net N$18: track 0.00 -> 2.54 mm
- net N$24: track 0.00 -> 2.54 mm
- net N$19: track 0.00 -> 2.54 mm
- net N$26: track 4.45 -> 6.02 mm
- net P1_5_3V: track 22.6 -> 21.2 mm
Other:
- board text added: "boh"
- board text added: "ch"
- board text added: "supplyframe"
- board text removed: "chain"
- board text removed: "layerOne 2016"
- board text removed: "supplyFrame.com"
